File: secs_q84 v2.brd (EAGLE design)
At the start: 78.4 x 58.4 mm, 65 parts, among them IC1 MAX203ECWP, IC2 REF3440TIDBVR, IC4 PIC18F47Q84-I_PT

Commit message: up
Parts:
- added 3.3V_PWR: 3.3V_PWR, pinhead:1X02
- added C16, C19: 0.1uf, rcl:C0805
- added C17, C18: 10uf, rcl:C0805
- added IC3: ADP151AUJZ-3.3-R7, ADP151AUJZ-3.3-R7:SOT95P280X100-5N
- added IC6: 74HC125D, 74HC125D:SOIC127P600X175-14N
- moved TP1 23.3 mm to (52.1, 54.6)
Connections:
- net 80VAN0 renamed 80VANA1
- net 80VAN1 renamed 80VANA2
- net AN0 renamed ANA0
- net RD5 renamed AND5
- net RE2 renamed SS_CS
- removed net AN1: ANALOG.1, IC4.20, R13.2, R3.1, R4.2, Z1.1
- removed net AN2: ANALOG.2, IC4.21, R14.2, R15.1, R16.1, Z2.1
- removed net AN4: ANALOG.4, IC4.23, R11.2, R12.2
- removed net AN5: ANALOG.5, IC4.24, R10.2, R2.2
- removed net PGD: EXT_IO.6, IC4.17, ICSP.4
- new net +3V3: 3.3V_PWR.2, C16.1, C17.1, IC3.5, IC6.14
- new net ANA1: ANALOG.1, IC4.20, R11.2, R12.2, R13.2, R3.1, R4.2, Z1.1
- new net ANA2: ANALOG.2, IC4.21, R10.2, R14.2, R15.1, R16.1, R2.2, Z2.1
- new net ANA4: ANALOG.4, IC4.23
- new net ANA5: ANALOG.5, IC4.24
- new net PGD_DAC1: EXT_IO.6, IC4.17, ICSP.4, SV1.2
- new net SCK2_OUT: IC6.6, SPI2.3
- new net SD02_OUT: IC6.3, SPI2.5
- new net SDI2_IN: IC6.12, SPI2.4
- new net SS2_OUT: IC6.8, SPI2.2
- net SCK2: now also IC6.5; no longer SPI2.3
- net SDI2: now also IC6.11; no longer SPI2.4
- net SDO2: now also IC6.2; no longer SPI2.5
- net SS2: now also IC6.9; no longer SPI2.2
- net VDD: now also C18.1, C19.1, IC3.1, IC3.3
- net VSS: now also 3.3V_PWR.1, C16.2, C17.2, C18.2, C19.2, IC3.2, IC6.1, IC6.10, IC6.13, IC6.4, IC6.7; no longer SV1.2
Routing:
- net ANA2: track 0.00 -> 136.5 mm, vias 0 -> 5
- net ANA1: track 0.00 -> 124.4 mm, vias 0 -> 5
- net AN1: track 110.2 -> 0.00 mm, vias 4 -> 0
- net AN2: track 102.4 -> 0.00 mm, vias 4 -> 0
- net PGD_DAC1: track 0.00 -> 89.9 mm, vias 0 -> 1
- net PGD: track 87.6 -> 0.00 mm, vias 1 -> 0
- net AN4: track 60.1 -> 0.00 mm, vias 2 -> 0
- net MCLR_SIG: track 79.9 -> 139.1 mm, vias 2 -> 0
- net AN5: track 52.6 -> 0.00 mm, vias 2 -> 0
- net ANA5: track 0.00 -> 50.4 mm, vias 0 -> 1
- net RC2: track 56.7 -> 11.3 mm
- net +3V3: track 0.00 -> 32.1 mm, vias 0 -> 2
- net ANA4: track 0.00 -> 30.4 mm, vias 0 -> 2
- net VSS: track 52.3 -> 23.0 mm, vias 8 -> 11
- net SS2: track 58.8 -> 31.2 mm, vias 1 -> 2
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
Commit message: pcb updates
Parts:
- added C20, C21: 0.1uf, rcl:C0805
- added C22: 10uf, rcl:C0805
- added IC5: MCZ33996EK, MCZ33996EK:SOP65P1030X265-33N
- added J1, J2: 87914-1016, 87914-1016:879141016
- added R20, R21, R22, R23, R24: 0ohm, rcl:R0805
- added R25: 1k, rcl:R0805
- moved B-NORM 10.9 mm to (77.5, 58.4)
- moved B-REV 10.2 mm to (88.9, 58.4)
- moved A+NORM 9.67 mm to (77.5, 55.9)
- moved A+REV 8.98 mm to (88.9, 55.9)
- moved C3 7.73 mm to (50.8, 35.6)
- moved R13 3.81 mm to (71.1, 68.6)
- moved R16 2.54 mm to (71.1, 71.1)
- moved TP2 2.54 mm to (96.5, 30.5)
- moved C11 2.54 mm to (50.8, 38.1)
- moved C6 1.27 mm to (71.1, 73.7)
Connections:
- removed net DEBUG1: EXT_IO.3, IC4.5, MISC_IO.7
- removed net RELAY0: IC4.25, MISC_IO.1
- new net MCZ_CS: IC4.25, IC5.14, MISC_IO.1
- new net MCZ_PWM: EXT_IO.3, IC4.5, IC5.30, MISC_IO.7
- new net N$10: R22.1, SPI2.4
- new net N$11: R23.1, SPI2.3
- new net N$12: R24.1, SPI2.2
- new net N$13: C20.1, IC5.27, R25.2
- new net N$14: IC5.1, J1.2
- new net N$15: IC5.2, J1.3
- new net N$16: IC5.4, J1.4
- new net N$17: IC5.5, J1.5
- new net N$18: IC5.12, J1.6
- new net N$19: IC5.13, J1.7
- new net N$20: IC5.15, J1.8
- new net N$21: IC5.16, J1.9
- new net N$22: IC5.32, J2.9
- new net N$23: IC5.31, J2.8
- new net N$24: IC5.29, J2.7
- new net N$25: IC5.28, J2.6
- new net N$26: IC5.21, J2.5
- new net N$27: IC5.20, J2.4
- new net N$28: IC5.18, J2.3
- new net N$29: IC5.17, J2.2
- new net N$8: R20.1, SPI2.6
- new net N$9: R21.1, SPI2.5
- net SCK1: now also IC5.11
- net SCK2_OUT: now also R23.2; no longer SPI2.3
- net SD02_OUT: now also R21.2; no longer SPI2.5
- net SDI1: now also DISPLAY.2, IC5.22
- net SDI2_IN: now also R22.2; no longer SPI2.4
- net SDO1: now also IC5.19
- net SPI2_REQ: now also R20.2; no longer SPI2.6
- net SS2_OUT: now also R24.2; no longer SPI2.2
- net VDD: now also C21.1, C22.1, IC5.3, IC5.6, R25.1
- net VSS: now also C20.2, C21.2, C22.2, IC5.10, IC5.23, IC5.24, IC5.25, IC5.26, IC5.33, IC5.7, IC5.8, IC5.9, J1.1, J1.10, J2.1, J2.10
Routing:
- net SDI1: track 21.3 -> 105.9 mm, vias 0 -> 3
- net MCZ_CS: track 0.00 -> 82.4 mm, vias 0 -> 2
- net MCZ_PWM: track 0.00 -> 74.9 mm, vias 0 -> 2
- net MCLR_SIG: track 139.1 -> 77.7 mm, vias 0 -> 3
- net DEBUG1: track 48.4 -> 0.00 mm, vias 1 -> 0
- net VDD: track 316.9 -> 359.3 mm, vias 11 -> 10
- net RS232RX: track 64.3 -> 98.8 mm, vias 3 -> 2
- net VSS: track 23.0 -> 49.1 mm, vias 11 -> 10
- net SDO1: track 83.2 -> 108.0 mm, vias 0 -> 3
- net RELAY0: track 24.1 -> 0.00 mm
- net N$14: track 0.00 -> 23.5 mm, vias 0 -> 1
- net N$16: track 0.00 -> 21.7 mm, vias 0 -> 1
- net N$28: track 0.00 -> 19.7 mm, vias 0 -> 1
- net ANA5: track 50.4 -> 32.2 mm
- net N$29: track 0.00 -> 18.1 mm, vias 0 -> 1
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
Commit message: cleaning up new PCB
Parts:
- added C23, C24, C26, C28: 0.1uf, rcl:C0805
- added C25: 1uf, rcl:C0805
- added C27: 10uf, rcl:C0805
- added IC7: TIC12400DCPR, TIC12400DCPR:SOP50P640X120-39N
- added J3: M20-8891045, M20-8891045:M208891045
- added R26, R27: 4.7k, rcl:R0805
- added VS_TIC_PWR: VS_TIC_PWR, pinhead:1X02
- moved C5 3.81 mm to (86.4, 33.0)
- moved Z2 2.54 mm to (77.5, 29.2)
Connections:
- removed net MISC: IC4.26, MISC_IO.2
- removed net PGC: EXT_IO.5, IC4.16, ICSP.5
- new net N$30: C23.1, IC7.23
- new net N$31: C25.1, IC7.22
- new net N$32: C24.1, IC7.20
- new net N$33: IC7.14, J3.3
- new net N$34: IC7.13, J3.2
- new net N$35: IC7.25, J3.4
- new net N$36: IC7.26, J3.5
- new net N$37: IC7.27, J3.6
- new net N$38: IC7.29, J3.7
- new net N$39: IC7.30, J3.8
- new net N$40: IC7.31, J3.9
- new net PGC_TICINT: EXT_IO.5, IC4.16, IC7.24, ICSP.5, R26.2
- new net TIC_CS: IC4.26, IC7.15, MISC_IO.2
- new net VS_TIC_24V: C26.1, C27.1, IC7.37, IC7.38, J3.10, VS_TIC_PWR.2
- net +3V3: now also R27.2
- net SCK1: now also IC7.16
- net SDI1: now also IC7.18
- net SDO1: now also IC7.17
- net SPI2_REQ: now also R27.1
- net VDD: now also C28.1, IC7.19, R26.1
- net VSS: now also C23.2, C24.2, C25.2, C26.2, C27.2, C28.2, IC7.21, IC7.28, IC7.39, IC7.9, J3.1, VS_TIC_PWR.1
Routing:
- net VS_TIC_24V: track 0.00 -> 98.0 mm, vias 0 -> 2
- net PGC_TICINT: track 0.00 -> 84.1 mm, vias 0 -> 4
- net N$40: track 0.00 -> 78.5 mm, vias 0 -> 3
- net N$37: track 0.00 -> 78.2 mm, vias 0 -> 3
- net N$39: track 0.00 -> 76.4 mm
- net PGC: track 74.9 -> 0.00 mm, vias 1 -> 0
- net N$38: track 0.00 -> 74.3 mm, vias 0 -> 2
- net N$36: track 0.00 -> 72.1 mm, vias 0 -> 2
- net N$35: track 0.00 -> 65.7 mm, vias 0 -> 2
- net TIC_CS: track 0.00 -> 61.9 mm, vias 0 -> 2
- net N$33: track 0.00 -> 52.6 mm, vias 0 -> 3
- net N$34: track 0.00 -> 52.3 mm, vias 0 -> 2
- net MCLR_SIG: track 77.7 -> 117.5 mm, vias 3 -> 1
- net PGD_DAC1: track 88.1 -> 120.8 mm
- net MISC: track 25.7 -> 0.00 mm
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
Commit message: up
Parts:
- added R28, R29: 400 ohm, rcl:R0805
- added TIC_DIGITAL: TIC_DIGITAL, con-lstb:MA04-1
- moved C21 3.81 mm to (82.5, 73.7), flipped to the top
- moved IC5 2.54 mm to (85.1, 66.0)
- moved R14 1.27 mm to (63.5, 27.9)
- moved R15 1.27 mm to (69.8, 27.9)
Connections:
- new net IN8D: R28.1, TIC_DIGITAL.2
- new net IN9D: R29.1, TIC_DIGITAL.3
- new net N$41: IC7.32, R28.2
- new net N$42: IC7.33, R29.2
- net VDD: now also TIC_DIGITAL.4
- net VSS: now also TIC_DIGITAL.1
Routing:
- net N$41: track 0.00 -> 64.2 mm
- net N$42: track 0.00 -> 50.0 mm, vias 0 -> 3
- net SDI1: track 97.5 -> 129.8 mm, vias 6 -> 4
- net PGD_DAC1: track 120.8 -> 91.7 mm
- net PGC_TICINT: track 84.1 -> 105.4 mm, vias 4 -> 3
- net N$37: track 78.2 -> 58.4 mm, vias 3 -> 2
- net ANA5: track 31.1 -> 50.0 mm, vias 0 -> 1
- net RLED: track 33.7 -> 16.1 mm
- net SDO2: track 56.9 -> 41.3 mm, vias 2 -> 4
- net MCLR_SIG: track 117.5 -> 103.9 mm, vias 1 -> 2
- net N$33: track 52.6 -> 65.9 mm, vias 3 -> 2
- net MCZ_CS: track 70.2 -> 83.3 mm, vias 3 -> 2
- net RS232RX: track 105.6 -> 92.9 mm, vias 1 -> 3
- net SDI2: track 70.8 -> 58.6 mm
- net IN8D: track 0.00 -> 11.8 mm
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
Commit message: up
Parts:
- added R30: 10k, rcl:R0805
Connections:
- net +3V3: now also R30.1
- net SS2_OUT: now also R30.2
Routing:
- net N$37: track 58.4 -> 107.0 mm, vias 2 -> 3
- net SS2_OUT: track 11.2 -> 43.0 mm, vias 1 -> 2
- net VDD: track 367.6 -> 342.8 mm
- net PGD_DAC1: track 91.7 -> 112.6 mm, vias 1 -> 0
- net CLOCKO: track 61.8 -> 41.4 mm, vias 1 -> 4
- net PGC_TICINT: track 105.4 -> 122.5 mm, vias 3 -> 2
- net SDI1: track 129.8 -> 113.3 mm
- net N$42: track 50.0 -> 65.2 mm, vias 3 -> 4
- net PC_RX2: track 47.0 -> 59.5 mm
- net N$35: track 75.0 -> 63.2 mm, vias 4 -> 2
- net VREF_4.1: track 46.6 -> 58.0 mm
- net N$40: track 89.2 -> 99.2 mm
- net ANC6: track 30.0 -> 39.6 mm
- net SCK1: track 106.4 -> 115.7 mm, vias 4 -> 3
- net N$39: track 80.4 -> 71.5 mm, vias 4 -> 3
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
Commit message: pcb order
Parts:
- moved F1 9.67 mm to (39.4, 25.4)
- moved ZENER 2.54 mm to (58.4, 66.0)
- moved R30 2.54 mm to (25.4, 71.1), flipped to the top
- moved DIG_ANA 1.27 mm to (31.8, 59.7)
- flipped C15 to the top
- flipped C18 to the top
- flipped C23 to the top
- flipped C24 to the top
- flipped C27 to the top
- flipped C6 to the top
- flipped R1 to the top
- flipped R13 to the top
- flipped R16 to the top
- flipped R19 to the top
- flipped R7 to the top
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Routing:
- net VSS: track 68.6 -> 112.8 mm, vias 10 -> 9
- net PGC_TICINT: track 122.5 -> 87.7 mm, vias 2 -> 3
- net N$38: track 69.8 -> 95.7 mm, vias 2 -> 3
- net ANA4: track 29.6 -> 54.7 mm, vias 0 -> 1
- net PGD_DAC1: track 112.6 -> 89.5 mm, vias 0 -> 1
- net N$36: track 75.9 -> 53.5 mm, vias 4 -> 2
- net N$40: track 99.2 -> 78.1 mm
- net MB_RX: track 39.9 -> 60.9 mm, vias 0 -> 3
- net PC_RX2: track 59.5 -> 39.2 mm, vias 1 -> 2
- net SS_CS: track 27.4 -> 47.0 mm, vias 0 -> 2
- net N$37: track 107.0 -> 126.4 mm, vias 3 -> 2
- net N$42: track 65.2 -> 83.6 mm, vias 4 -> 3
- net SCK1: track 115.7 -> 97.4 mm
- net SDI1: track 113.3 -> 96.3 mm, vias 4 -> 3
- net SS2_OUT: track 43.0 -> 28.0 mm
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