File: secs_q84 v2.brd (EAGLE design)
At the start: 78.4 x 58.4 mm, 100 parts, among them IC1 MAX203ECWP, IC2 REF3440TIDBVR, IC3 ADP151AUJZ-3.3-R7, IC4 PIC18F47Q84-I_PT, IC5 MCZ33996EK, IC6 74HC125D, IC7 TIC12400DCPR, J1 87914-1016, J2 87914-1016

Commit message: v1.1 update
Parts:
- removed J1, J2: 87914-1016, 87914-1016:879141016
- added DO1, DO2: 87914-1016, 87914-1016:879141016
- added F2: 0805L075WR, 0805L075WR:FUSC2114X125N
Connections:
- removed net TIC0: IC7.13, TIC_INPUT_0_7.2
- removed net TIC1: IC7.14, TIC_INPUT_0_7.3
- new net 24V_IN: F2.1, VS_TIC_PWR.2
- new net TIC10: IC7.34, TIC_INPUT_0_7.2
- new net TIC11: IC7.35, TIC_INPUT_0_7.3
- net MO0: now also DO1.1; no longer J1.2
- net MO1: now also DO1.2; no longer J1.3
- net MO10: now also DO2.3; no longer J2.4
- net MO11: now also DO2.4; no longer J2.5
- net MO12: now also DO2.5; no longer J2.6
- net MO13: now also DO2.6; no longer J2.7
- net MO14: now also DO2.7; no longer J2.8
- net MO15: now also DO2.8; no longer J2.9
- net MO2: now also DO1.3; no longer J1.4
- net MO3: now also DO1.4; no longer J1.5
- net MO4: now also DO1.5; no longer J1.6
- net MO5: now also DO1.6; no longer J1.7
- net MO6: now also DO1.7; no longer J1.8
- net MO7: now also DO1.8; no longer J1.9
- net MO8: now also DO2.1; no longer J2.2
- net MO9: now also DO2.2; no longer J2.3
- net VDD: now also DO1.9, DO2.9
- net VSS: now also DO1.10, DO2.10; no longer J1.1, J1.10, J2.1, J2.10
- net VS_TIC_24V: now also F2.2; no longer VS_TIC_PWR.2
Routing:
- net TIC11: track 0.00 -> 63.4 mm
- net TIC10: track 0.00 -> 62.8 mm, vias 0 -> 2
- net TIC1: track 54.2 -> 0.00 mm, vias 4 -> 0
- net TIC0: track 48.2 -> 0.00 mm
- net VDD: track 355.8 -> 388.2 mm
- net MO1: track 9.26 -> 19.4 mm
- net MO0: track 16.1 -> 23.9 mm
- net VSS: track 112.8 -> 117.9 mm
- net 24V_IN: track 0.00 -> 4.79 mm
- net MO15: track 13.6 -> 18.3 mm
- net MO3: track 7.89 -> 11.1 mm
- net MO13: track 14.2 -> 16.8 mm, vias 1 -> 2
- net MO7: track 13.1 -> 10.9 mm
- net MO5: track 7.91 -> 6.08 mm
- net MO9: track 13.0 -> 14.6 mm
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Other:
- board text added: "+"
- board text added: "Linux BMC slave Q84 V1.10"
- board text removed: "Linux BMS slave Q84 V1.10"

Commit message: up
Parts:
- removed TIC_INPUT_0_7: M20-8891045, M20-8891045:M208891045
- added DIO_RESET: dio reset, pinhead:1X01
- added SHORT_VV: short_vv, jumper:SJ
- added TIC0_7, TIC16_23, TIC8_15: 87914-1016, 87914-1016:879141016
- moved IC7 50.6 mm to (68.6, 17.8)
- moved C24 46.7 mm to (78.7, 15.2), flipped to the bottom, turned to 270 degrees
- moved C23 44.4 mm to (78.7, 20.3), flipped to the bottom, turned to 270 degrees
- moved C25 38.1 mm to (78.7, 24.1)
- moved C28 37.0 mm to (57.1, 24.1)
- moved R26 35.1 mm to (53.3, 20.3)
- moved TIC_DIGITAL 30.5 mm to (35.6, 15.2)
- moved DO2 26.9 mm to (97.8, 62.2), turned to 0 degrees
- moved TTL_SERIAL 13.7 mm to (35.6, 19.1)
- moved C6 12.7 mm to (83.8, 73.7)
- moved C21 11.4 mm to (71.1, 73.7)
- moved DO1 10.2 mm to (97.8, 69.8), turned to 0 degrees
- moved IC5 9.67 mm to (76.2, 62.2)
- moved C12 9.67 mm to (48.3, 20.3), turned to 180 degrees
- moved R16 9.16 mm to (76.2, 63.5)
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Connections:
- removed net N$13: C20.1, IC5.27, R25.2
- new net DIO_RST: C20.1, DIO_RESET.1, IC5.27, R25.2
- new net TIC0: IC7.13, TIC0_7.1
- new net TIC1: IC7.14, TIC0_7.2
- new net TIC12: IC7.36, TIC8_15.5
- new net TIC13: IC7.1, TIC8_15.6
- new net TIC14: IC7.2, TIC8_15.7
- new net TIC15: IC7.3, TIC8_15.8
- new net TIC16: IC7.4, TIC16_23.1
- new net TIC17: IC7.5, TIC16_23.2
- new net TIC18: IC7.6, TIC16_23.3
- new net TIC19: IC7.7, TIC16_23.4
- new net TIC20: IC7.8, TIC16_23.5
- new net TIC21: IC7.10, TIC16_23.6
- new net TIC22: IC7.11, TIC16_23.7
- new net TIC23: IC7.12, TIC16_23.8
- net GND: no longer LED4.C
- net TIC10: now also TIC8_15.3; no longer TIC_INPUT_0_7.2
- net TIC11: now also TIC8_15.4; no longer TIC_INPUT_0_7.3
- net TIC2: now also TIC0_7.3; no longer TIC_INPUT_0_7.4
- net TIC3: now also TIC0_7.4; no longer TIC_INPUT_0_7.5
- net TIC4: now also TIC0_7.5; no longer TIC_INPUT_0_7.6
- net TIC5: now also TIC0_7.6; no longer TIC_INPUT_0_7.7
- net TIC6: now also TIC0_7.7; no longer TIC_INPUT_0_7.8
- net TIC7: now also TIC0_7.8; no longer TIC_INPUT_0_7.9
- net TIC8: now also TIC8_15.1
- net TIC9: now also TIC8_15.2
- net VCC: now also SHORT_VV.2; no longer R19.1
- net VDD: now also R19.1, SHORT_VV.1
- net VSS: now also LED4.C, TIC0_7.10, TIC16_23.10, TIC8_15.10; no longer TIC_INPUT_0_7.1
- net VS_TIC_24V: now also TIC0_7.9, TIC16_23.9, TIC8_15.9; no longer TIC_INPUT_0_7.10
Routing:
- net TIC4: track 126.4 -> 13.5 mm, vias 2 -> 1
- net SCK1: track 97.4 -> 202.5 mm
- net SDO1: track 114.8 -> 196.7 mm, vias 3 -> 4
- net TIC5: track 95.7 -> 13.9 mm, vias 3 -> 1
- net VS_TIC_24V: track 103.2 -> 173.5 mm, vias 3 -> 4
- net TIC6: track 81.8 -> 15.6 mm, vias 2 -> 1
- net TIC9: track 83.6 -> 18.8 mm, vias 3 -> 2
- net DIO_RST: track 0.00 -> 61.6 mm, vias 0 -> 3
- net TIC7: track 78.1 -> 17.8 mm, vias 2 -> 1
- net TIC11: track 63.4 -> 6.87 mm, vias 0 -> 1
- net TIC10: track 62.8 -> 11.0 mm, vias 2 -> 1
- net TIC2: track 57.3 -> 10.7 mm, vias 4 -> 1
- net SDO2: track 43.6 -> 90.0 mm
- net TIC8: track 67.7 -> 23.0 mm
- net SDI1: track 96.3 -> 139.2 mm, vias 3 -> 6
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Other:
- board size 78.4 x 58.4 mm -> 78.4 x 69.8 mm
- board text added: "Linux BMC slave Q84 V1.20"
- board text removed: "Linux BMC slave Q84 V1.10"

Commit message: PCB updates:wq
Parts:
- added C29: 10uf, rcl:C0805
- added INT_RESET: reset, jumper:SJ
Connections:
- net MCZ_PWM: now also INT_RESET.2
- net R_RESET: now also C29.1, INT_RESET.1
- net VSS: now also C29.2
Routing:
- net MCZ_PWM: track 63.7 -> 72.5 mm
- net R_RESET: track 86.5 -> 89.1 mm
Changed lines of the file:
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@@
 <attribute name="VALUE" x="35.9601" y="25.4" size="0.02" layer="27"/>
+</element>
+<element name="C29" library="rcl" library_urn="urn:adsk.eagle:library:334" package="C0805" package3d_urn="urn:adsk.eagle:package:23617/2" value="10uf" x="48.26" y="44.45" smashed="yes" rot="MR0">
+<attribute name="NAME" x="49.53" y="45.72" size="1.27" layer="26" rot="MR0"/>
+<attribute name="POPULARITY" value="63" x="48.26" y="44.45" size="1.778" layer="28" rot="MR0" display="off"/>
+<attribute name="SPICEPREFIX" value="C" x="48.26" y="44.45" size="1.778" layer="28" rot="MR0" display="off"/>
+<attribute name="VALUE" x="49.53" y="41.91" size="1.27" layer="28" rot="MR0"/>
+</element>
+<element name="INT_RESET" library="jumper" library_urn="urn:adsk.eagle:library:252" package="SJ" package3d_urn="urn:adsk.eagle:package:15471/1" value="reset" x="57.15" y="69.85" smashed="yes">
+<attribute name="NAME" x="54.229" y="67.183" size="1.27" layer="25" ratio="10"/>
+<attribute name="POPULARITY" value="33" x="57.15" y="69.85" size="1.778" layer="27" display="off"/>
+<attribute name="VALUE" x="57.5501" y="69.85" size="0.02" layer="27"/>
 </element>
 </elements>
@@
 <wire x1="71.518" y1="18.28" x2="74.43" y2="18.28" width="0.254" layer="16"/>
 <wire x1="74.43" y1="18.28" x2="74.93" y2="17.78" width="0.254" layer="16"/>
+<contactref element="C29" pad="2"/>
 </signal>
 <signal name="CPU_CLK">
@@
 <wire x1="59.6646" y1="76.2" x2="59.69" y2="76.2" width="0.1524" layer="1"/>
 <wire x1="49.2252" y1="44.1198" x2="49.2252" y2="41.91" width="0.1524" layer="16"/>
-<wire x1="51.2826" y1="46.1772" x2="49.2252" y2="44.1198" width="0.1524" layer="16"/>
+<wire x1="51.2826" y1="46.1772" x2="49.3776" y2="44.2722" width="0.1524" layer="16"/>
+<wire x1="49.3776" y1="44.2722" x2="49.2252" y2="44.1198" width="0.1524" layer="16"/>
 <wire x1="51.2826" y1="47.1678" x2="51.2826" y2="46.1772" width="0.1524" layer="1"/>
 <wire x1="54.864" y1="50.7492" x2="51.2826" y2="47.1678" width="0.1524" layer="1"/>
@@
 <wire x1="24.6126" y1="74.9046" x2="24.638" y2="74.93" width="0.1524" layer="1"/>
 <wire x1="55.5498" y1="72.39" x2="57.47" y2="72.39" width="0.1524" layer="1"/>
-<wire x1="52.7304" y1="69.5706" x2="55.5498" y2="72.39" width="0.1524" layer="1"/>
+<wire x1="52.7304" y1="69.5706" x2="54.7116" y2="71.5518" width="0.1524" layer="1"/>
+<wire x1="54.7116" y1="71.5518" x2="55.5498" y2="72.39" width="0.1524" layer="1"/>
 <wire x1="50.8254" y1="69.5706" x2="52.7304" y2="69.5706" width="0.1524" layer="1"/>
 <wire x1="49.7586" y1="68.5038" x2="50.8254" y2="69.5706" width="0.1524" layer="1"/>
@@
 <via x="40.1574" y="61.1124" extent="1-16" drill="0.35"/>
 <via x="49.7586" y="68.5038" extent="1-16" drill="0.35"/>
+<contactref element="C29" pad="1"/>
+<wire x1="49.3776" y1="44.2722" x2="49.2252" y2="44.4246" width="0.1524" layer="16"/>
+<wire x1="49.2252" y1="44.4246" x2="49.21" y2="44.45" width="0.1524" layer="16"/>
+<contactref element="INT_RESET" pad="1"/>
+<wire x1="54.7116" y1="71.5518" x2="56.388" y2="69.8754" width="0.1524" layer="1"/>
+<wire x1="56.388" y1="69.8754" x2="56.388" y2="69.85" width="0.1524" layer="1"/>
 </signal>
 <signal name="ANA0">
@@
 <via x="39.0144" y="42.3672" extent="1-16" drill="0.35"/>
 <via x="43.6626" y="62.7888" extent="1-16" drill="0.35"/>
+<contactref element="INT_RESET" pad="2"/>
+<wire x1="57.912" y1="69.342" x2="57.912" y2="69.85" width="0.1524" layer="1"/>
+<wire x1="52.07" y1="63.5" x2="57.912" y2="69.342" width="0.1524" layer="1"/>
 </signal>
 <signal name="SDI2">

Commit message: up
Parts:
- removed INT_RESET: reset, jumper:SJ
- added INT_RESET1: int_reset, pinhead:1X02
Connections:
- net MCZ_PWM: now also INT_RESET1.2; no longer INT_RESET.2
- net R_RESET: now also INT_RESET1.1; no longer INT_RESET.1
Routing:
- net VSS: vias 12 -> 17
Other:
- board text added: "Linux BMC slave Q84 V1.22"
- board text removed: "Linux BMC slave Q84 V1.20"
Changed lines of the file:
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@@
 <wire x1="100" y1="80" x2="21.59" y2="80" width="0" layer="20"/>
 <wire x1="21.59" y1="80" x2="21.59" y2="10.16" width="0" layer="20"/>
-<text x="99.06" y="33.02" size="1.27" layer="1" font="vector" ratio="15" distance="70" rot="R90">Linux BMC slave Q84 V1.20</text>
+<text x="99.06" y="33.02" size="1.27" layer="1" font="vector" ratio="15" distance="70" rot="R90">Linux BMC slave Q84 V1.22</text>
 <polygon width="0.1524" layer="41">
 <vertex x="44.45" y="41.91"/>
@@
 <attribute name="VALUE" x="49.53" y="41.91" size="1.27" layer="28" rot="MR0"/>
 </element>
-<element name="INT_RESET" library="jumper" library_urn="urn:adsk.eagle:library:252" package="SJ" package3d_urn="urn:adsk.eagle:package:15471/1" value="reset" x="57.15" y="69.85" smashed="yes">
-<attribute name="NAME" x="54.229" y="67.183" size="1.27" layer="25" ratio="10"/>
-<attribute name="POPULARITY" value="33" x="57.15" y="69.85" size="1.778" layer="27" display="off"/>
-<attribute name="VALUE" x="57.5501" y="69.85" size="0.02" layer="27"/>
+<element name="INT_RESET1" library="pinhead" library_urn="urn:adsk.eagle:library:325" package="1X02" package3d_urn="urn:adsk.eagle:package:22435/2" value="int_reset" x="57.15" y="69.85" smashed="yes">
+<attribute name="NAME" x="53.2638" y="66.5988" size="1.27" layer="25" ratio="10"/>
+<attribute name="POPULARITY" value="98" x="57.15" y="69.85" size="1.778" layer="27" display="off"/>
+<attribute name="VALUE" x="54.61" y="66.675" size="1.27" layer="27"/>
 </element>
 </elements>
@@
 <wire x1="87.63" y1="69.7992" x2="86.487" y2="68.6562" width="0.254" layer="2"/>
 <wire x1="87.63" y1="69.7992" x2="87.63" y2="69.85" width="0.254" layer="2"/>
-<wire x1="59.3598" y1="66.675" x2="59.3598" y2="72.39" width="0.254" layer="1"/>
-<wire x1="58.4454" y1="65.7606" x2="59.3598" y2="66.675" width="0.254" layer="1"/>
-<wire x1="59.3598" y1="72.39" x2="59.37" y2="72.39" width="0.254" layer="1"/>
-<wire x1="58.4454" y1="65.7606" x2="58.42" y2="65.7" width="0.254" layer="1"/>
 <wire x1="80.1624" y1="63.8556" x2="80.9244" y2="63.8556" width="0.254" layer="16"/>
 <wire x1="79.5528" y1="64.4652" x2="80.1624" y2="63.8556" width="0.254" layer="16"/>
@@
 <wire x1="56.388" y1="38.1" x2="55.7022" y2="38.7858" width="0.254" layer="15"/>
 <wire x1="53.4924" y1="48.2346" x2="53.4162" y2="48.3108" width="0.254" layer="15"/>
-<wire x1="56.8452" y1="64.0842" x2="58.3692" y2="65.6082" width="0.254" layer="1"/>
 <wire x1="56.8452" y1="53.2638" x2="56.8452" y2="64.0842" width="0.254" layer="15"/>
 <wire x1="53.4924" y1="49.911" x2="56.8452" y2="53.2638" width="0.254" layer="15"/>
 <wire x1="53.4924" y1="48.387" x2="53.4924" y2="49.911" width="0.254" layer="15"/>
-<wire x1="58.3692" y1="65.6082" x2="58.42" y2="65.7" width="0.254" layer="1"/>
 <wire x1="53.4924" y1="48.387" x2="53.4162" y2="48.3108" width="0.254" layer="15"/>
 <wire x1="38.2524" y1="42.1386" x2="31.7754" y2="42.1386" width="0.254" layer="2"/>
@@
 <via x="63.8556" y="30.4038" extent="1-16" drill="0.35"/>
 <via x="56.8452" y="64.0842" extent="1-16" drill="0.35"/>
+<wire x1="59.436" y1="71.0946" x2="59.436" y2="72.3138" width="0.254" layer="1"/>
+<wire x1="59.5122" y1="71.0184" x2="59.436" y2="71.0946" width="0.254" layer="1"/>
+<wire x1="59.5122" y1="66.8274" x2="59.5122" y2="71.0184" width="0.254" layer="1"/>
+<wire x1="59.436" y1="72.3138" x2="59.37" y2="72.39" width="0.254" layer="1"/>
+<wire x1="58.5216" y1="65.8368" x2="59.5122" y2="66.8274" width="0.254" layer="1"/>
+<wire x1="58.5216" y1="65.8368" x2="58.42" y2="65.7" width="0.254" layer="1"/>
+<wire x1="58.42" y1="65.7" x2="58.42" y2="65.659" width="0.254" layer="1"/>
+<wire x1="58.42" y1="65.659" x2="56.8452" y2="64.0842" width="0.254" layer="1"/>
 </signal>
 <signal name="VSS" class="1">
@@
 <wire x1="74.43" y1="18.28" x2="74.93" y2="17.78" width="0.254" layer="16"/>
 <contactref element="C29" pad="2"/>
+<via x="82.55" y="25.4" extent="1-16" drill="0.35" locked="yes"/>
+<via x="86.36" y="25.4" extent="1-16" drill="0.35" locked="yes"/>
+<via x="90.17" y="25.4" extent="1-16" drill="0.35" locked="yes"/>
+<via x="86.36" y="29.21" extent="1-16" drill="0.35" locked="yes"/>
+<via x="86.36" y="31.75" extent="1-16" drill="0.35" locked="yes"/>
 </signal>
 <signal name="CPU_CLK">
@@
 <wire x1="24.6126" y1="74.9046" x2="24.638" y2="74.93" width="0.1524" layer="1"/>
 <wire x1="55.5498" y1="72.39" x2="57.47" y2="72.39" width="0.1524" layer="1"/>
-<wire x1="52.7304" y1="69.5706" x2="54.7116" y2="71.5518" width="0.1524" layer="1"/>
-<wire x1="54.7116" y1="71.5518" x2="55.5498" y2="72.39" width="0.1524" layer="1"/>
+<wire x1="52.7304" y1="69.5706" x2="54.4449" y2="71.2851" width="0.1524" layer="1"/>
+<wire x1="54.4449" y1="71.2851" x2="55.5498" y2="72.39" width="0.1524" layer="1"/>
 <wire x1="50.8254" y1="69.5706" x2="52.7304" y2="69.5706" width="0.1524" layer="1"/>
 <wire x1="49.7586" y1="68.5038" x2="50.8254" y2="69.5706" width="0.1524" layer="1"/>
@@
 <wire x1="49.3776" y1="44.2722" x2="49.2252" y2="44.4246" width="0.1524" layer="16"/>
 <wire x1="49.2252" y1="44.4246" x2="49.21" y2="44.45" width="0.1524" layer="16"/>
-<contactref element="INT_RESET" pad="1"/>
-<wire x1="54.7116" y1="71.5518" x2="56.388" y2="69.8754" width="0.1524" layer="1"/>
-<wire x1="56.388" y1="69.8754" x2="56.388" y2="69.85" width="0.1524" layer="1"/>
+<contactref element="INT_RESET1" pad="1"/>
+<wire x1="54.4449" y1="71.2851" x2="55.88" y2="69.85" width="0.1524" layer="1"/>
 </signal>
 <signal name="ANA0">
@@
 <via x="39.0144" y="42.3672" extent="1-16" drill="0.35"/>
 <via x="43.6626" y="62.7888" extent="1-16" drill="0.35"/>
-<contactref element="INT_RESET" pad="2"/>
-<wire x1="57.912" y1="69.342" x2="57.912" y2="69.85" width="0.1524" layer="1"/>
-<wire x1="52.07" y1="63.5" x2="57.912" y2="69.342" width="0.1524" layer="1"/>
+<contactref element="INT_RESET1" pad="2"/>
+<wire x1="52.07" y1="63.5" x2="58.42" y2="69.85" width="0.1524" layer="1"/>
 </signal>
 <signal name="SDI2">

Commit message: up uuuppp#	modified:   secs_q84 v2.b#5
Parts:
- removed IC4: PIC18F47Q84-I_PT, PIC18F47Q84-I_PT:QFP80P1200X1200X120-44N
- removed R27: 4.7k, rcl:R0805
- added IC8: PIC18F57Q84-I_PT, PIC18F57Q84-I_PT:QFP50P900X900X120-49N
- added R31: 4.7k, rcl:R0805
- moved TIC8_15 43.2 mm to (115.6, 26.7)
- moved TIC16_23 22.9 mm to (115.6, 17.8)
- moved PVP_0 20.4 mm to (110.5, 39.4)
- moved TP2 19.0 mm to (81.3, 38.1)
- moved DO2 15.5 mm to (113.0, 59.7)
- moved DIO_RESET 15.3 mm to (86.4, 38.1)
- moved DO1 15.2 mm to (113.0, 69.8)
- moved C22 14.2 mm to (90.2, 68.6)
- moved R13 14.2 mm to (90.2, 63.5)
- moved C20 14.2 mm to (90.2, 66.0)
- moved R16 14.2 mm to (90.2, 61.0)
- moved IC5 14.0 mm to (90.2, 63.5)
- moved C6 3.59 mm to (86.4, 71.1)
- moved R1 2.84 mm to (77.5, 71.1)
Connections:
- net +3V3: now also R31.2; no longer R27.2
- net ANA0: now also IC8.21; no longer IC4.19
- net ANA1: now also IC8.22; no longer IC4.20
- net ANA2: now also IC8.23; no longer IC4.21
- net ANA4: now also IC8.25; no longer IC4.23
- net ANA5: now also IC8.26; no longer IC4.24
- net ANC6: now also IC8.48; no longer IC4.44
- net ANC7: now also IC8.1; no longer IC4.1
- net AND5: now also IC8.3; no longer IC4.3
- net CLOCKO: now also IC8.33; no longer IC4.31
- net CPU_CLK: now also IC8.32; no longer IC4.30
- net CS: now also IC8.45; no longer IC4.41
- net DLED: now also IC8.11, IC8.2; no longer IC4.11, IC4.2
- net MB_RX: now also IC8.34; no longer IC4.32
- net MB_TX: now also IC8.35; no longer IC4.35
- net MCLR_SIG: now also IC8.20; no longer IC4.18
- net MCZ_CS: now also IC8.27; no longer IC4.25
- net MCZ_PWM: now also IC8.5; no longer IC4.5
- net MLED: now also IC8.9; no longer IC4.9
- net PC_RX2: now also IC8.42; no longer IC4.38
- net PC_TX2: now also IC8.4; no longer IC4.4
- net PGC_TICINT: now also IC8.18; no longer IC4.16
- net PGD_DAC1: now also IC8.19; no longer IC4.17
- net RLED: now also IC8.10; no longer IC4.10
- net SCK1: now also IC8.41; no longer IC4.37
- net SCK2: now also IC8.44; no longer IC4.40
- net SDI1: now also IC8.46; no longer IC4.42
- net SDI2: now also IC8.17; no longer IC4.15
- net SDO1: now also IC8.47; no longer IC4.43
- net SDO2: now also IC8.16; no longer IC4.14
- net SPI2_REQ: now also IC8.8, R31.1; no longer IC4.8, R27.1
- net SS2: now also IC8.43; no longer IC4.39
- net SS_CS: now also IC8.29; no longer IC4.27
- net TIC_CS: now also IC8.28; no longer IC4.26
- net TP1_TEST_SIG: now also IC8.40; no longer IC4.36
- net VDD: now also IC8.30, IC8.7; no longer IC4.28, IC4.7
- net VREF_4.1: now also IC8.24; no longer IC4.22
- net VSS: now also IC8.31, IC8.49, IC8.6; no longer IC4.29, IC4.6
Routing:
- net TIC9: track 18.8 -> 85.5 mm, vias 2 -> 1
- net SDO1: track 196.7 -> 145.9 mm
- net TIC8: track 23.0 -> 72.5 mm
- net TIC11: track 6.87 -> 53.1 mm
- net TIC10: track 11.0 -> 54.1 mm, vias 1 -> 2
- net TIC13: track 5.50 -> 44.4 mm, vias 0 -> 1
- net SCK1: track 202.5 -> 164.1 mm
- net TIC12: track 9.20 -> 47.3 mm, vias 1 -> 2
- net MCLR_SIG: track 117.7 -> 80.7 mm, vias 1 -> 2
- net TIC23: track 14.8 -> 48.5 mm
- net TIC15: track 8.62 -> 37.7 mm
- net TIC19: track 21.3 -> 48.0 mm
- net TIC14: track 13.0 -> 39.0 mm
- net TIC16: track 23.7 -> 48.9 mm
- net TIC20: track 17.2 -> 40.9 mm
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Other:
- board size 78.4 x 69.8 mm -> 97.5 x 69.8 mm
