File: secs_q84 v2.sch (EAGLE design)
At the start: 66 parts, among them IC1 MAX203ECWP, IC2 REF3440TIDBVR, IC4 PIC18F47Q84-I_PT

Commit message: up
Parts:
- removed CANBUS: CANBUS, con-lstb:MA06-1
- removed CANBUS_TERM: 120 ohm, rcl:R-US_R0805
- added SPI2: SPI2, con-lstb:MA06-1
- DIG_ANA: value Digtal -> Digtal/Analog
- renumbered DIGITAL to DIG_ANA
Connections:
- net RD7 renamed DEBUG1
- net RELAY renamed RELAY0
- net UC_RX renamed ANC7
- net UC_TX renamed ANC6
- removed net CANRX: CANBUS.2, CANBUS_TERM.1, IC4.RB0
- removed net CANTX: CANBUS.3, CANBUS_TERM.2, IC4.RB4
- removed net DB0: DIG_ANA.1, IC4.RD1
- removed net DB1: DIG_ANA.2, IC4.RD2
- removed net DERE: CANBUS.4, IC4.RC2, TP1.TP
- removed net RB5: EXT_IO.4, IC4.RB5, MISC_IO.6
- new net RC2: IC4.RC2, TP1.TP
- new net SCK2: DIG_ANA.2, IC4.RD2, SPI2.3
- new net SDI2: EXT_IO.4, IC4.RB5, MISC_IO.6, SPI2.4
- new net SDO2: IC4.RB4, SPI2.5
- new net SPI2_REQ: IC4.RB0, SPI2.6
- new net SS2: DIG_ANA.1, IC4.RD1, SPI2.2
- net VDD: no longer CANBUS.5
- net VSS: now also SPI2.1; no longer CANBUS.1

Commit message: up
Parts:
- added 3.3V_PWR: 3.3V_PWR, pinhead:PINHD-1X2
- added C16, C19: 0.1uf, rcl:C-USC0805
- added C17, C18: 10uf, rcl:C-USC0805
- added IC3: ADP151AUJZ-3.3-R7, ADP151AUJZ-3.3-R7:ADP151AUJZ-3.3-R7
- added IC6: 74HC125D, 74HC125D:74HC125D
Connections:
- net 80VAN0 renamed 80VANA1
- net 80VAN1 renamed 80VANA2
- net AN0 renamed ANA0
- net RD5 renamed AND5
- net RE2 renamed SS_CS
- removed net AN1: ANALOG.1, IC4.RA1, R13.2, R3.1, R4.2, Z1.K
- removed net AN2: ANALOG.2, IC4.RA2, R14.2, R15.1, R16.1, Z2.K
- removed net AN4: ANALOG.4, IC4.RA4, R11.2, R12.2
- removed net AN5: ANALOG.5, IC4.RA5, R10.2, R2.2
- removed net PGD: EXT_IO.6, IC4.ICSPDAT/RB7, ICSP.4
- new net +3V3: 3.3V_PWR.2, C16.1, C17.1, IC3.VOUT, IC6.VCC
- new net ANA1: ANALOG.1, IC4.RA1, R11.2, R12.2, R13.2, R3.1, R4.2, Z1.K
- new net ANA2: ANALOG.2, IC4.RA2, R10.2, R14.2, R15.1, R16.1, R2.2, Z2.K
- new net ANA4: ANALOG.4, IC4.RA4
- new net ANA5: ANALOG.5, IC4.RA5
- new net PGD_DAC1: EXT_IO.6, IC4.ICSPDAT/RB7, ICSP.4, SV1.2
- new net SCK2_OUT: IC6.2Y, SPI2.3
- new net SD02_OUT: IC6.1Y, SPI2.5
- new net SDI2_IN: IC6.4A, SPI2.4
- new net SS2_OUT: IC6.3Y, SPI2.2
- net SCK2: now also IC6.2A; no longer SPI2.3
- net SDI2: now also IC6.4Y; no longer SPI2.4
- net SDO2: now also IC6.1A; no longer SPI2.5
- net SS2: now also IC6.3A; no longer SPI2.2
- net VDD: now also C18.1, C19.1, IC3.EN, IC3.VIN
- net VSS: now also 3.3V_PWR.1, C16.2, C17.2, C18.2, C19.2, IC3.GND, IC6.1!G, IC6.2!G, IC6.3!G, IC6.4!G, IC6.GND; no longer SV1.2

Commit message: pcb updates
Parts:
- added C20, C21: 0.1uf, rcl:C-USC0805
- added C22: 10uf, rcl:C-USC0805
- added IC5: MCZ33996EK, MCZ33996EK:MCZ33996EK
- added J1, J2: 87914-1016, 87914-1016:87914-1016
- added R20, R21, R22, R23, R24: 0ohm, rcl:R-US_R0805
- added R25: 1k, rcl:R-US_R0805
Connections:
- removed net DEBUG1: EXT_IO.3, IC4.RD7, MISC_IO.7
- removed net RELAY0: IC4.RE0, MISC_IO.1
- new net MCZ_CS: IC4.RE0, IC5.!CS, MISC_IO.1
- new net MCZ_PWM: EXT_IO.3, IC4.RD7, IC5.PWM, MISC_IO.7
- new net N$10: R22.1, SPI2.4
- new net N$11: R23.1, SPI2.3
- new net N$12: R24.1, SPI2.2
- new net N$13: C20.1, IC5.!RST, R25.2
- new net N$14: IC5.OUT0, J1.2
- new net N$15: IC5.OUT1, J1.3
- new net N$16: IC5.OUT2, J1.4
- new net N$17: IC5.OUT3, J1.5
- new net N$18: IC5.OUT4, J1.6
- new net N$19: IC5.OUT5, J1.7
- new net N$20: IC5.OUT6, J1.8
- new net N$21: IC5.OUT7, J1.9
- new net N$22: IC5.OUT15, J2.9
- new net N$23: IC5.OUT14, J2.8
- new net N$24: IC5.OUT13, J2.7
- new net N$25: IC5.OUT12, J2.6
- new net N$26: IC5.OUT11, J2.5
- new net N$27: IC5.OUT10, J2.4
- new net N$28: IC5.OUT9, J2.3
- new net N$29: IC5.OUT8, J2.2
- new net N$8: R20.1, SPI2.6
- new net N$9: R21.1, SPI2.5
- net SCK1: now also IC5.SCLK
- net SCK2_OUT: now also R23.2; no longer SPI2.3
- net SD02_OUT: now also R21.2; no longer SPI2.5
- net SDI1: now also DISPLAY.2, IC5.SO
- net SDI2_IN: now also R22.2; no longer SPI2.4
- net SDO1: now also IC5.SI
- net SPI2_REQ: now also R20.2; no longer SPI2.6
- net SS2_OUT: now also R24.2; no longer SPI2.2
- net VDD: now also C21.1, C22.1, IC5.SOPWR, IC5.VPWR, R25.1
- net VSS: now also C20.2, C21.2, C22.2, IC5.EP, IC5.GND_1, IC5.GND_2, IC5.GND_3, IC5.GND_4, IC5.GND_5, IC5.GND_6, IC5.GND_7, IC5.GND_8, J1.1, J1.10, J2.1, J2.10

Commit message: cleaning up new PCB
Parts:
- added C23, C24, C26, C28: 0.1uf, rcl:C-USC0805
- added C25: 1uf, rcl:C-USC0805
- added C27: 10uf, rcl:C-USC0805
- added IC7: TIC12400DCPR, TIC12400DCPR:TIC12400DCPR
- added J3: M20-8891045, M20-8891045:M20-8891045
- added R26, R27: 4.7k, rcl:R-US_R0805
- added VS_TIC_PWR: VS_TIC_PWR, pinhead:PINHD-1X2
Connections:
- removed net MISC: IC4.RE1, MISC_IO.2
- removed net PGC: EXT_IO.5, IC4.ICSPCLK/RB6, ICSP.5
- new net N$30: C23.1, IC7.CAP_D
- new net N$31: C25.1, IC7.CAP_PRE
- new net N$32: C24.1, IC7.CAP_A
- new net N$33: IC7.IN1, J3.3
- new net N$34: IC7.IN0, J3.2
- new net N$35: IC7.IN2, J3.4
- new net N$36: IC7.IN3, J3.5
- new net N$37: IC7.IN4, J3.6
- new net N$38: IC7.IN5, J3.7
- new net N$39: IC7.IN6, J3.8
- new net N$40: IC7.IN7, J3.9
- new net PGC_TICINT: EXT_IO.5, IC4.ICSPCLK/RB6, IC7.!INT, ICSP.5, R26.2
- new net TIC_CS: IC4.RE1, IC7.!CS, MISC_IO.2
- new net VS_TIC_24V: C26.1, C27.1, IC7.VS_1, IC7.VS_2, J3.10, VS_TIC_PWR.2
- net +3V3: now also R27.2
- net SCK1: now also IC7.SCLK
- net SDI1: now also IC7.SO
- net SDO1: now also IC7.SI
- net SPI2_REQ: now also R27.1
- net VDD: now also C28.1, IC7.VDD, R26.1
- net VSS: now also C23.2, C24.2, C25.2, C26.2, C27.2, C28.2, IC7.AGND, IC7.DGND, IC7.EP, IC7.RESET, J3.1, VS_TIC_PWR.1

Commit message: up
Parts:
- added R28, R29: 400 ohm, rcl:R-US_R0805
- added TIC_DIGITAL: TIC_DIGITAL, con-lstb:MA04-1
Connections:
- new net IN8D: R28.1, TIC_DIGITAL.2
- new net IN9D: R29.1, TIC_DIGITAL.3
- new net N$41: IC7.IN8, R28.2
- new net N$42: IC7.IN9, R29.2
- net VDD: now also TIC_DIGITAL.4
- net VSS: now also TIC_DIGITAL.1
Changed lines of the file:
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@@
 <class number="0" name="default" width="0" drill="0">
 </class>
-<class number="1" name="icurrent" width="0.3048" drill="0">
+<class number="1" name="icurrent" width="0.254" drill="0">
 </class>
-<class number="2" name="ocurrent" width="0.254" drill="0">
+<class number="2" name="ocurrent" width="0.2032" drill="0">
 </class>
 </classes>
@@
 <part name="C28" library="rcl" library_urn="urn:adsk.eagle:library:334" deviceset="C-US" device="C0805" package3d_urn="urn:adsk.eagle:package:23617/2" value="0.1uf"/>
 <part name="VSS70" library="supply1" library_urn="urn:adsk.eagle:library:371" deviceset="VSS" device=""/>
+<part name="R28" library="rcl" library_urn="urn:adsk.eagle:library:334" deviceset="R-US_" device="R0805" package3d_urn="urn:adsk.eagle:package:23553/2" value="400 ohm"/>
+<part name="R29" library="rcl" library_urn="urn:adsk.eagle:library:334" deviceset="R-US_" device="R0805" package3d_urn="urn:adsk.eagle:package:23553/2" value="400 ohm"/>
+<part name="TIC_DIGITAL" library="con-lstb" library_urn="urn:adsk.eagle:library:162" deviceset="MA04-1" device="" package3d_urn="urn:adsk.eagle:package:8337/1" value="TIC_DIGITAL"/>
+<part name="VSS71" library="supply1" library_urn="urn:adsk.eagle:library:371" deviceset="VSS" device=""/>
+<part name="VDD23" library="supply1" library_urn="urn:adsk.eagle:library:371" deviceset="VDD" device=""/>
 </parts>
 <sheets>
@@
 <attribute name="VALUE" x="-38.1" y="-137.16" size="1.778" layer="96" rot="R180"/>
 </instance>
+<instance part="R28" gate="G$1" x="30.48" y="-91.44" smashed="yes" rot="R180">
+<attribute name="NAME" x="34.29" y="-92.9386" size="1.778" layer="95" rot="R180"/>
+<attribute name="VALUE" x="39.37" y="-93.218" size="1.778" layer="96" rot="R180"/>
+</instance>
+<instance part="R29" gate="G$1" x="30.48" y="-88.9" smashed="yes" rot="R180">
+<attribute name="NAME" x="29.21" y="-85.3186" size="1.778" layer="95" rot="R180"/>
+<attribute name="VALUE" x="34.29" y="-85.598" size="1.778" layer="96" rot="R180"/>
+</instance>
+<instance part="TIC_DIGITAL" gate="1" x="114.3" y="-121.92" smashed="yes">
+<attribute name="VALUE" x="113.03" y="-132.08" size="1.778" layer="96"/>
+<attribute name="NAME" x="113.03" y="-116.078" size="1.778" layer="95"/>
+</instance>
+<instance part="VSS71" gate="G$1" x="121.92" y="-129.54" smashed="yes">
+<attribute name="VALUE" x="124.46" y="-134.62" size="1.778" layer="96" rot="R180"/>
+</instance>
+<instance part="VDD23" gate="G$1" x="121.92" y="-116.84" smashed="yes">
+<attribute name="VALUE" x="124.46" y="-111.76" size="1.778" layer="96" rot="R180"/>
+</instance>
 </instances>
 <busses>
@@
 <junction x="38.1" y="-111.76"/>
 </segment>
+<segment>
+<pinref part="TIC_DIGITAL" gate="1" pin="4"/>
+<pinref part="VDD23" gate="G$1" pin="VDD"/>
+<junction x="121.92" y="-119.38"/>
+</segment>
 </net>
 <net name="VSS" class="1">
@@
 <junction x="-40.64" y="-129.54"/>
 </segment>
+<segment>
+<pinref part="TIC_DIGITAL" gate="1" pin="1"/>
+<pinref part="VSS71" gate="G$1" pin="VSS"/>
+<junction x="121.92" y="-127"/>
+</segment>
 </net>
 <net name="CPU_CLK" class="0">
@@
 </segment>
 </net>
+<net name="N$41" class="0">
+<segment>
+<pinref part="IC7" gate="G$1" pin="IN8"/>
+<wire x1="5.08" y1="-91.44" x2="25.4" y2="-91.44" width="0.1524" layer="91"/>
+<junction x="5.08" y="-91.44"/>
+<junction x="25.4" y="-91.44"/>
+<pinref part="R28" gate="G$1" pin="2"/>
+<label x="10.16" y="-91.44" size="1.778" layer="95"/>
+</segment>
+</net>
+<net name="N$42" class="0">
+<segment>
+<pinref part="IC7" gate="G$1" pin="IN9"/>
+<wire x1="5.08" y1="-88.9" x2="25.4" y2="-88.9" width="0.1524" layer="91"/>
+<junction x="5.08" y="-88.9"/>
+<junction x="25.4" y="-88.9"/>
+<pinref part="R29" gate="G$1" pin="2"/>
+<label x="10.16" y="-88.9" size="1.778" layer="95"/>
+</segment>
+</net>
+<net name="IN8D" class="0">
+<segment>
+<pinref part="R28" gate="G$1" pin="1"/>
+<wire x1="35.56" y1="-91.44" x2="48.26" y2="-91.44" width="0.1524" layer="91"/>
+<junction x="35.56" y="-91.44"/>
+<junction x="48.26" y="-91.44"/>
+<label x="38.1" y="-91.44" size="1.778" layer="95"/>
+</segment>
+<segment>
+<wire x1="121.92" y1="-124.46" x2="127" y2="-124.46" width="0.1524" layer="91"/>
+<pinref part="TIC_DIGITAL" gate="1" pin="2"/>
+<junction x="127" y="-124.46"/>
+<junction x="121.92" y="-124.46"/>
+<label x="132.08" y="-124.46" size="1.778" layer="95"/>
+</segment>
+</net>
+<net name="IN9D" class="0">
+<segment>
+<pinref part="R29" gate="G$1" pin="1"/>
+<wire x1="35.56" y1="-88.9" x2="48.26" y2="-88.9" width="0.1524" layer="91"/>
+<junction x="35.56" y="-88.9"/>
+<junction x="48.26" y="-88.9"/>
+<label x="40.64" y="-88.9" size="1.778" layer="95"/>
+</segment>
+<segment>
+<wire x1="121.92" y1="-121.92" x2="127" y2="-121.92" width="0.1524" layer="91"/>
+<pinref part="TIC_DIGITAL" gate="1" pin="3"/>
+<junction x="127" y="-121.92"/>
+<junction x="121.92" y="-121.92"/>
+<label x="132.08" y="-121.92" size="1.778" layer="95"/>
+</segment>
+</net>

Commit message: up
Parts:
- added R30: 10k, rcl:R-US_R0805
Connections:
- net +3V3: now also R30.1
- net SS2_OUT: now also R30.2
Changed lines of the file:
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@@
 <part name="VSS71" library="supply1" library_urn="urn:adsk.eagle:library:371" deviceset="VSS" device=""/>
 <part name="VDD23" library="supply1" library_urn="urn:adsk.eagle:library:371" deviceset="VDD" device=""/>
+<part name="R30" library="rcl" library_urn="urn:adsk.eagle:library:334" deviceset="R-US_" device="R0805" package3d_urn="urn:adsk.eagle:package:23553/2" value="10k"/>
+<part name="+3V5" library="supply1" library_urn="urn:adsk.eagle:library:371" deviceset="+3V3" device=""/>
 </parts>
 <sheets>
@@
 <instance part="VDD23" gate="G$1" x="121.92" y="-116.84" smashed="yes">
 <attribute name="VALUE" x="124.46" y="-111.76" size="1.778" layer="96" rot="R180"/>
+</instance>
+<instance part="R30" gate="G$1" x="144.78" y="10.16" smashed="yes" rot="R90">
+<attribute name="NAME" x="143.2814" y="6.35" size="1.778" layer="95" rot="R90"/>
+<attribute name="VALUE" x="148.082" y="6.35" size="1.778" layer="96" rot="R90"/>
+</instance>
+<instance part="+3V5" gate="G$1" x="152.4" y="7.62" smashed="yes">
+<attribute name="VALUE" x="152.4" y="10.16" size="1.778" layer="96"/>
 </instance>
 </instances>
@@
 <junction x="160.02" y="15.24"/>
 <label x="144.78" y="15.24" size="1.778" layer="95"/>
+<pinref part="R30" gate="G$1" pin="2"/>
 </segment>
 </net>
@@
 <junction x="170.18" y="-20.32"/>
 </segment>
-</net>
+<segment>
+<pinref part="R30" gate="G$1" pin="1"/>
+<pinref part="+3V5" gate="G$1" pin="+3V3"/>
+<wire x1="144.78" y1="5.08" x2="152.4" y2="5.08" width="0.1524" layer="91"/>
+<junction x="144.78" y="5.08"/>
+<junction x="152.4" y="5.08"/>
+</segment>
+</net>

Commit message: up
Connections:
- removed net SCK2_OUT: IC6.2Y, R23.2
- removed net SS2_OUT: IC6.3Y, R24.2, R30.2
- new net SCK2_IN: IC6.2A, R23.2
- new net SS2_IN: IC6.3A, R24.2, R30.2
- net SCK2: now also IC6.2Y; no longer IC6.2A
- net SS2: now also IC6.3Y; no longer IC6.3A
Other:
- note added: "5/6 and 8/9 pins swapped as a fix"
Changed lines of the file:
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@@
 <sheet>
 <plain>
+<text x="332.74" y="-20.32" size="1.778" layer="91">5/6 and 8/9 pins swapped as a fix</text>
 </plain>
 <instances>
@@
 </instance>
 <instance part="IC3" gate="G$1" x="335.28" y="-25.4" smashed="yes">
-<attribute name="NAME" x="359.41" y="-17.78" size="1.778" layer="95" align="center-left"/>
-<attribute name="VALUE" x="359.41" y="-20.32" size="1.778" layer="96" align="center-left"/>
+<attribute name="NAME" x="346.71" y="-35.56" size="1.778" layer="95" align="center-left"/>
+<attribute name="VALUE" x="341.63" y="-38.1" size="1.778" layer="96" align="center-left"/>
 </instance>
 <instance part="IC6" gate="G$1" x="335.28" y="0" smashed="yes">
@@
 </instance>
 <instance part="VSS45" gate="G$1" x="332.74" y="-15.24" smashed="yes" rot="R270">
-<attribute name="VALUE" x="330.2" y="-12.7" size="1.778" layer="96" rot="R180"/>
+<attribute name="VALUE" x="330.2" y="-15.24" size="1.778" layer="96" rot="R180"/>
 </instance>
 <instance part="VSS46" gate="G$1" x="363.22" y="-10.16" smashed="yes" rot="R90">
@@
 </instance>
 <instance part="VDD13" gate="G$1" x="335.28" y="-22.86" smashed="yes">
-<attribute name="VALUE" x="332.74" y="-20.32" size="1.778" layer="96" rot="R180"/>
+<attribute name="VALUE" x="330.2" y="-22.86" size="1.778" layer="96" rot="R180"/>
 </instance>
 <instance part="VDD15" gate="G$1" x="335.28" y="-33.02" smashed="yes" rot="R180">
@@
 </segment>
 <segment>
-<wire x1="373.38" y1="-12.7" x2="360.68" y2="-12.7" width="0.1524" layer="91"/>
-<pinref part="IC6" gate="G$1" pin="3A"/>
-<junction x="360.68" y="-12.7"/>
-<junction x="373.38" y="-12.7"/>
-<label x="363.22" y="-12.7" size="1.778" layer="95"/>
+<wire x1="373.38" y1="-15.24" x2="360.68" y2="-15.24" width="0.1524" layer="91"/>
+<pinref part="IC6" gate="G$1" pin="3Y"/>
+<junction x="373.38" y="-15.24"/>
+<junction x="360.68" y="-15.24"/>
+<label x="363.22" y="-15.24" size="1.778" layer="95"/>
 </segment>
 </net>
@@
 </segment>
 <segment>
-<wire x1="322.58" y1="-10.16" x2="335.28" y2="-10.16" width="0.1524" layer="91"/>
-<pinref part="IC6" gate="G$1" pin="2A"/>
-<junction x="335.28" y="-10.16"/>
-<junction x="322.58" y="-10.16"/>
-<label x="325.12" y="-10.16" size="1.778" layer="95"/>
+<wire x1="322.58" y1="-12.7" x2="335.28" y2="-12.7" width="0.1524" layer="91"/>
+<pinref part="IC6" gate="G$1" pin="2Y"/>
+<junction x="335.28" y="-12.7"/>
+<junction x="322.58" y="-12.7"/>
+<label x="325.12" y="-12.7" size="1.778" layer="95"/>
 </segment>
 </net>
@@
 </segment>
 </net>
-<net name="SCK2_OUT" class="0">
-<segment>
-<wire x1="320.04" y1="-12.7" x2="335.28" y2="-12.7" width="0.1524" layer="91"/>
-<pinref part="IC6" gate="G$1" pin="2Y"/>
-<junction x="335.28" y="-12.7"/>
-<junction x="320.04" y="-12.7"/>
-<label x="322.58" y="-12.7" size="1.778" layer="95"/>
-</segment>
+<net name="SCK2_IN" class="0">
 <segment>
 <wire x1="144.78" y1="17.78" x2="160.02" y2="17.78" width="0.1524" layer="91"/>
@@
 <label x="147.32" y="17.78" size="1.778" layer="95"/>
 </segment>
-</net>
-<net name="SS2_OUT" class="0">
-<segment>
-<wire x1="360.68" y1="-15.24" x2="375.92" y2="-15.24" width="0.1524" layer="91"/>
-<pinref part="IC6" gate="G$1" pin="3Y"/>
-<junction x="360.68" y="-15.24"/>
-<junction x="375.92" y="-15.24"/>
-<label x="363.22" y="-15.24" size="1.778" layer="95"/>
-</segment>
+<segment>
+<wire x1="320.04" y1="-10.16" x2="335.28" y2="-10.16" width="0.1524" layer="91"/>
+<pinref part="IC6" gate="G$1" pin="2A"/>
+<junction x="335.28" y="-10.16"/>
+<junction x="320.04" y="-10.16"/>
+<label x="322.58" y="-10.16" size="1.778" layer="95"/>
+</segment>
+</net>
+<net name="SS2_IN" class="0">
 <segment>
 <wire x1="144.78" y1="15.24" x2="160.02" y2="15.24" width="0.1524" layer="91"/>
@@
 <pinref part="R30" gate="G$1" pin="2"/>
 </segment>
-</net>
+<segment>
+<wire x1="360.68" y1="-12.7" x2="375.92" y2="-12.7" width="0.1524" layer="91"/>
+<pinref part="IC6" gate="G$1" pin="3A"/>
+<junction x="375.92" y="-12.7"/>
+<junction x="360.68" y="-12.7"/>
+<label x="363.22" y="-12.7" size="1.778" layer="95"/>
+</segment>
+</net>

Commit message: up
Connections:
- net 80VANA1 renamed 80VANA4
- net 80VANA2 renamed 80VANA5
- net ANA1: no longer R11.2, R12.2
- net ANA2: no longer R10.2, R2.2
- net ANA4: now also R11.2, R12.2
- net ANA5: now also R10.2, R2.2
Changed lines of the file:
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@@
 <pinref part="Z1" gate="G$1" pin="K"/>
-</segment>
-<segment>
-<pinref part="R11" gate="G$1" pin="2"/>
-<pinref part="R12" gate="G$1" pin="2"/>
-<wire x1="-15.24" y1="48.26" x2="-17.78" y2="48.26" width="0.1524" layer="91"/>
-<junction x="-17.78" y="48.26"/>
-<junction x="-15.24" y="48.26"/>
-<label x="-12.7" y="48.26" size="1.778" layer="95"/>
 </segment>
 </net>
@@
 <pinref part="Z2" gate="G$1" pin="K"/>
 </segment>
-<segment>
-<pinref part="R2" gate="G$1" pin="2"/>
-<pinref part="R10" gate="G$1" pin="2"/>
-<wire x1="-5.08" y1="50.8" x2="-15.24" y2="50.8" width="0.1524" layer="91"/>
-<junction x="-5.08" y="50.8"/>
-<junction x="-15.24" y="50.8"/>
-<label x="-10.16" y="50.8" size="1.778" layer="95"/>
-</segment>
 </net>
 <net name="PC_RX2" class="0">
@@
 <label x="241.3" y="-27.94" size="1.778" layer="95"/>
 </segment>
+<segment>
+<pinref part="R11" gate="G$1" pin="2"/>
+<pinref part="R12" gate="G$1" pin="2"/>
+<wire x1="-15.24" y1="48.26" x2="-17.78" y2="48.26" width="0.1524" layer="91"/>
+<junction x="-15.24" y="48.26"/>
+<junction x="-17.78" y="48.26"/>
+<label x="-15.24" y="48.26" size="1.778" layer="95"/>
+</segment>
 </net>
 <net name="ANA5" class="0">
@@
 <junction x="246.38" y="-25.4"/>
 <label x="236.22" y="-25.4" size="1.778" layer="95"/>
+</segment>
+<segment>
+<pinref part="R2" gate="G$1" pin="2"/>
+<pinref part="R10" gate="G$1" pin="2"/>
+<wire x1="-5.08" y1="50.8" x2="-15.24" y2="50.8" width="0.1524" layer="91"/>
+<junction x="-5.08" y="50.8"/>
+<junction x="-15.24" y="50.8"/>
+<label x="-5.08" y="50.8" size="1.778" layer="95"/>
 </segment>
 </net>
@@
 </segment>
 </net>
-<net name="80VANA1" class="0">
+<net name="80VANA4" class="0">
 <segment>
 <pinref part="ANALOG" gate="1" pin="6"/>
@@
 </segment>
 </net>
-<net name="80VANA2" class="0">
+<net name="80VANA5" class="0">
 <segment>
 <pinref part="R2" gate="G$1" pin="1"/>
