File: secs_q84 v2.sch (EAGLE design)
At the start: 116 parts, among them IC1 MAX203ECWP, IC2 REF3440TIDBVR, IC3 ADP151AUJZ-3.3-R7, IC4 ADM3095EBRZ, IC5 MCZ33996EK, IC6 74HC125D, IC7 TIC12400DCPR, IC8 PIC18F57Q84-I_PT

Commit message: up
Parts:
- added AUX_IO: AUX_IO, con-lstb:MA06-1
Connections:
- new net RF4: AUX_IO.3, IC8.RF4
- new net RF5: AUX_IO.4, IC8.RF5
- new net RF6: AUX_IO.5, IC8.RF6
- new net RF7: AUX_IO.6, IC8.RF7
- net VDD: now also AUX_IO.2
- net VSS: now also AUX_IO.1
Changed lines of the file:
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@@
 <part name="DE3" library="jumper" library_urn="urn:adsk.eagle:library:252" deviceset="SJ" device="" package3d_urn="urn:adsk.eagle:package:15471/1" value="DE3"/>
 <part name="TXDE3" library="jumper" library_urn="urn:adsk.eagle:library:252" deviceset="SJ" device="" package3d_urn="urn:adsk.eagle:package:15471/1" value="TXDE3"/>
+<part name="AUX_IO" library="con-lstb" library_urn="urn:adsk.eagle:library:162" deviceset="MA06-1" device="" package3d_urn="urn:adsk.eagle:package:8340/1" value="AUX_IO"/>
+<part name="VDD31" library="supply1" library_urn="urn:adsk.eagle:library:371" deviceset="VDD" device=""/>
+<part name="VSS83" library="supply1" library_urn="urn:adsk.eagle:library:371" deviceset="VSS" device=""/>
 </parts>
 <sheets>
@@
 <attribute name="VALUE" x="204.47" y="-35.56" size="1.778" layer="96" rot="R270"/>
 </instance>
+<instance part="AUX_IO" gate="1" x="220.98" y="-180.34" smashed="yes">
+<attribute name="VALUE" x="219.71" y="-193.04" size="1.778" layer="96"/>
+<attribute name="NAME" x="219.71" y="-171.958" size="1.778" layer="95"/>
+</instance>
+<instance part="VDD31" gate="G$1" x="231.14" y="-185.42" smashed="yes" rot="R270">
+<attribute name="VALUE" x="238.76" y="-185.42" size="1.778" layer="96" rot="R180"/>
+</instance>
+<instance part="VSS83" gate="G$1" x="231.14" y="-187.96" smashed="yes" rot="R90">
+<attribute name="VALUE" x="233.68" y="-190.5" size="1.778" layer="96"/>
+</instance>
 </instances>
 <busses>
@@
 <junction x="274.32" y="-30.48"/>
 </segment>
+<segment>
+<pinref part="AUX_IO" gate="1" pin="2"/>
+<pinref part="VDD31" gate="G$1" pin="VDD"/>
+<junction x="228.6" y="-185.42"/>
+</segment>
 </net>
 <net name="VSS" class="1">
@@
 <junction x="276.86" y="2.54"/>
 </segment>
+<segment>
+<pinref part="AUX_IO" gate="1" pin="1"/>
+<pinref part="VSS83" gate="G$1" pin="VSS"/>
+<junction x="228.6" y="-187.96"/>
+</segment>
 </net>
 <net name="CPU_CLK" class="0">
@@
 </segment>
 </net>
+<net name="RF4" class="0">
+<segment>
+<pinref part="IC8" gate="G$1" pin="RF4"/>
+<wire x1="254" y1="-152.4" x2="241.3" y2="-152.4" width="0.1524" layer="91"/>
+<junction x="254" y="-152.4"/>
+<junction x="241.3" y="-152.4"/>
+<label x="243.84" y="-152.4" size="1.778" layer="95"/>
+</segment>
+<segment>
+<wire x1="241.3" y1="-182.88" x2="228.6" y2="-182.88" width="0.1524" layer="91"/>
+<pinref part="AUX_IO" gate="1" pin="3"/>
+<junction x="228.6" y="-182.88"/>
+<junction x="241.3" y="-182.88"/>
+<label x="231.14" y="-182.88" size="1.778" layer="95"/>
+</segment>
+</net>
+<net name="RF7" class="0">
+<segment>
+<pinref part="IC8" gate="G$1" pin="RF7"/>
+<wire x1="266.7" y1="-180.34" x2="266.7" y2="-193.04" width="0.1524" layer="91"/>
+<junction x="266.7" y="-180.34"/>
+<junction x="266.7" y="-193.04"/>
+<label x="266.7" y="-190.5" size="1.778" layer="95" rot="R90"/>
+</segment>
+<segment>
+<wire x1="228.6" y1="-175.26" x2="241.3" y2="-175.26" width="0.1524" layer="91"/>
+<pinref part="AUX_IO" gate="1" pin="6"/>
+<junction x="228.6" y="-175.26"/>
+<junction x="241.3" y="-175.26"/>
+<label x="231.14" y="-175.26" size="1.778" layer="95"/>
+</segment>
+</net>
+<net name="RF6" class="0">
+<segment>
+<pinref part="IC8" gate="G$1" pin="RF6"/>
+<wire x1="264.16" y1="-180.34" x2="264.16" y2="-193.04" width="0.1524" layer="91"/>
+<junction x="264.16" y="-180.34"/>
+<junction x="264.16" y="-193.04"/>
+<label x="264.16" y="-190.5" size="1.778" layer="95" rot="R90"/>
+</segment>
+<segment>
+<wire x1="228.6" y1="-177.8" x2="241.3" y2="-177.8" width="0.1524" layer="91"/>
+<pinref part="AUX_IO" gate="1" pin="5"/>
+<junction x="228.6" y="-177.8"/>
+<junction x="241.3" y="-177.8"/>
+<label x="231.14" y="-177.8" size="1.778" layer="95"/>
+</segment>
+</net>
+<net name="RF5" class="0">
+<segment>
+<pinref part="IC8" gate="G$1" pin="RF5"/>
+<wire x1="261.62" y1="-180.34" x2="261.62" y2="-193.04" width="0.1524" layer="91"/>
+<junction x="261.62" y="-180.34"/>
+<junction x="261.62" y="-193.04"/>
+<label x="261.62" y="-190.5" size="1.778" layer="95" rot="R90"/>
+</segment>
+<segment>
+<wire x1="228.6" y1="-180.34" x2="241.3" y2="-180.34" width="0.1524" layer="91"/>
+<pinref part="AUX_IO" gate="1" pin="4"/>
+<junction x="228.6" y="-180.34"/>
+<junction x="241.3" y="-180.34"/>
+<label x="231.14" y="-180.34" size="1.778" layer="95"/>
+</segment>
+</net>

Commit message: up
Parts:
- added C32, C33, C34, C35: 0.1uf, rcl:C-USC0603
- added GLORY_24: GLORY_24, pinhead:PINHD-1X2
Connections:
- net RF4: now also C35.1
- net RF5: now also C32.1
- net RF6: now also C33.1
- net RF7: now also C34.1
- net VSS: now also C32.2, C33.2, C34.2, C35.2
- net VS_TIC_24V: now also GLORY_24.1, GLORY_24.2
Changed lines of the file:
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@@
 <part name="VDD31" library="supply1" library_urn="urn:adsk.eagle:library:371" deviceset="VDD" device=""/>
 <part name="VSS83" library="supply1" library_urn="urn:adsk.eagle:library:371" deviceset="VSS" device=""/>
+<part name="GLORY_24" library="pinhead" library_urn="urn:adsk.eagle:library:325" deviceset="PINHD-1X2" device="" package3d_urn="urn:adsk.eagle:package:22435/2" value="GLORY_24"/>
+<part name="C32" library="rcl" library_urn="urn:adsk.eagle:library:334" deviceset="C-US" device="C0603" package3d_urn="urn:adsk.eagle:package:23616/2" value="0.1uf"/>
+<part name="C33" library="rcl" library_urn="urn:adsk.eagle:library:334" deviceset="C-US" device="C0603" package3d_urn="urn:adsk.eagle:package:23616/2" value="0.1uf"/>
+<part name="C34" library="rcl" library_urn="urn:adsk.eagle:library:334" deviceset="C-US" device="C0603" package3d_urn="urn:adsk.eagle:package:23616/2" value="0.1uf"/>
+<part name="C35" library="rcl" library_urn="urn:adsk.eagle:library:334" deviceset="C-US" device="C0603" package3d_urn="urn:adsk.eagle:package:23616/2" value="0.1uf"/>
+<part name="VSS84" library="supply1" library_urn="urn:adsk.eagle:library:371" deviceset="VSS" device=""/>
+<part name="VSS85" library="supply1" library_urn="urn:adsk.eagle:library:371" deviceset="VSS" device=""/>
+<part name="VSS86" library="supply1" library_urn="urn:adsk.eagle:library:371" deviceset="VSS" device=""/>
+<part name="VSS87" library="supply1" library_urn="urn:adsk.eagle:library:371" deviceset="VSS" device=""/>
 </parts>
 <sheets>
@@
 </instance>
 <instance part="VSS22" gate="G$1" x="38.1" y="-53.34" smashed="yes">
-<attribute name="VALUE" x="40.64" y="-58.42" size="1.778" layer="96" rot="R180"/>
+<attribute name="VALUE" x="40.64" y="-55.88" size="1.778" layer="96" rot="R180"/>
 </instance>
 <instance part="VSS23" gate="G$1" x="27.94" y="-53.34" smashed="yes">
-<attribute name="VALUE" x="30.48" y="-58.42" size="1.778" layer="96" rot="R180"/>
+<attribute name="VALUE" x="22.86" y="-53.34" size="1.778" layer="96" rot="R180"/>
 </instance>
 <instance part="MISC_IO" gate="1" x="-15.24" y="10.16" smashed="yes">
@@
 </instance>
 <instance part="VSS35" gate="G$1" x="33.02" y="-53.34" smashed="yes">
-<attribute name="VALUE" x="35.56" y="-58.42" size="1.778" layer="96" rot="R180"/>
+<attribute name="VALUE" x="30.48" y="-55.88" size="1.778" layer="96" rot="R180"/>
 </instance>
 <instance part="R_RESET" gate="G$1" x="-33.02" y="78.74" smashed="yes" rot="R180">
@@
 <attribute name="VALUE" x="233.68" y="-190.5" size="1.778" layer="96"/>
 </instance>
+<instance part="GLORY_24" gate="G$1" x="45.72" y="-60.96" smashed="yes" rot="R180">
+<attribute name="NAME" x="57.15" y="-56.515" size="1.778" layer="95" rot="R180"/>
+<attribute name="VALUE" x="54.61" y="-53.34" size="1.778" layer="96" rot="R180"/>
+</instance>
+<instance part="C32" gate="G$1" x="261.62" y="-195.58" smashed="yes">
+<attribute name="NAME" x="262.636" y="-194.945" size="1.778" layer="95"/>
+<attribute name="VALUE" x="262.636" y="-199.771" size="1.778" layer="96"/>
+</instance>
+<instance part="C33" gate="G$1" x="264.16" y="-203.2" smashed="yes">
+<attribute name="NAME" x="265.176" y="-202.565" size="1.778" layer="95"/>
+<attribute name="VALUE" x="265.176" y="-207.391" size="1.778" layer="96"/>
+</instance>
+<instance part="C34" gate="G$1" x="266.7" y="-195.58" smashed="yes">
+<attribute name="NAME" x="267.716" y="-194.945" size="1.778" layer="95"/>
+<attribute name="VALUE" x="267.716" y="-199.771" size="1.778" layer="96"/>
+</instance>
+<instance part="C35" gate="G$1" x="241.3" y="-154.94" smashed="yes">
+<attribute name="NAME" x="242.316" y="-154.305" size="1.778" layer="95"/>
+<attribute name="VALUE" x="242.316" y="-159.131" size="1.778" layer="96"/>
+</instance>
+<instance part="VSS84" gate="G$1" x="241.3" y="-162.56" smashed="yes">
+<attribute name="VALUE" x="238.76" y="-165.1" size="1.778" layer="96" rot="R270"/>
+</instance>
+<instance part="VSS85" gate="G$1" x="259.08" y="-200.66" smashed="yes" rot="R270">
+<attribute name="VALUE" x="256.54" y="-198.12" size="1.778" layer="96" rot="R180"/>
+</instance>
+<instance part="VSS86" gate="G$1" x="269.24" y="-200.66" smashed="yes" rot="R90">
+<attribute name="VALUE" x="271.78" y="-203.2" size="1.778" layer="96"/>
+</instance>
+<instance part="VSS87" gate="G$1" x="264.16" y="-210.82" smashed="yes">
+<attribute name="VALUE" x="261.62" y="-213.36" size="1.778" layer="96" rot="R270"/>
+</instance>
 </instances>
 <busses>
@@
 <junction x="228.6" y="-187.96"/>
 </segment>
+<segment>
+<pinref part="C35" gate="G$1" pin="2"/>
+<pinref part="VSS84" gate="G$1" pin="VSS"/>
+<junction x="241.3" y="-160.02"/>
+</segment>
+<segment>
+<pinref part="C32" gate="G$1" pin="2"/>
+<pinref part="VSS85" gate="G$1" pin="VSS"/>
+<junction x="261.62" y="-200.66"/>
+</segment>
+<segment>
+<pinref part="C34" gate="G$1" pin="2"/>
+<pinref part="VSS86" gate="G$1" pin="VSS"/>
+<junction x="266.7" y="-200.66"/>
+</segment>
+<segment>
+<pinref part="C33" gate="G$1" pin="2"/>
+<pinref part="VSS87" gate="G$1" pin="VSS"/>
+<junction x="264.16" y="-208.28"/>
+</segment>
 </net>
 <net name="CPU_CLK" class="0">
@@
 <label x="195.58" y="-172.72" size="1.778" layer="95"/>
 </segment>
+<segment>
+<wire x1="48.26" y1="-60.96" x2="55.88" y2="-60.96" width="0.1524" layer="91"/>
+<pinref part="GLORY_24" gate="G$1" pin="2"/>
+<junction x="48.26" y="-60.96"/>
+<junction x="55.88" y="-60.96"/>
+<label x="27.94" y="-60.96" size="1.778" layer="95"/>
+</segment>
+<segment>
+<wire x1="48.26" y1="-63.5" x2="55.88" y2="-63.5" width="0.1524" layer="91"/>
+<pinref part="GLORY_24" gate="G$1" pin="1"/>
+<junction x="48.26" y="-63.5"/>
+<junction x="55.88" y="-63.5"/>
+<label x="27.94" y="-63.5" size="1.778" layer="95"/>
+</segment>
 </net>
 <net name="TIC2" class="0">
@@
 <junction x="241.3" y="-152.4"/>
 <label x="243.84" y="-152.4" size="1.778" layer="95"/>
+<pinref part="C35" gate="G$1" pin="1"/>
 </segment>
 <segment>
@@
 <junction x="266.7" y="-193.04"/>
 <label x="266.7" y="-190.5" size="1.778" layer="95" rot="R90"/>
+<pinref part="C34" gate="G$1" pin="1"/>
 </segment>
 <segment>
@@
 <junction x="264.16" y="-193.04"/>
 <label x="264.16" y="-190.5" size="1.778" layer="95" rot="R90"/>
+<pinref part="C33" gate="G$1" pin="1"/>
+<wire x1="264.16" y1="-200.66" x2="264.16" y2="-193.04" width="0.1524" layer="91"/>
+<junction x="264.16" y="-200.66"/>
 </segment>
 <segment>
@@
 <junction x="261.62" y="-193.04"/>
 <label x="261.62" y="-190.5" size="1.778" layer="95" rot="R90"/>
+<pinref part="C32" gate="G$1" pin="1"/>
 </segment>
 <segment>

Commit message: add FM80 interface
Parts:
- added C36: 0.1uf, rcl:C-USC0603
- added FM_RS: FM_RS, jumper:SJ
- added JMP1: 0R-JUMPA, jump-0r-smd:0R-JUMPA
- added MATE: MATE, con-lstb:MA04-1
- added OK1, OK2: 4N25SM, optocoupler:4N25SM
- added R34, R35: 2.2k, rcl:R-US_R0805
- added R36: 1k, rcl:R-US_R0805
- added R37: 470, rcl:R-US_R0805
Connections:
- removed net VS_TIC_24V: C26.1, C27.1, F2.2, GLORY_24.1, GLORY_24.2, IC7.VS_1, IC7.VS_2, TIC0_7.9, TIC16_23.9, TIC8_15.9
- new net 0V: MATE.2, R34.2, R35.1
- new net FM80_24: MATE.1, OK2.COL
- new net FM_RX: MATE.4, OK1.A
- new net FM_TX: MATE.3, OK2.EMI, R35.2
- new net MC_TIC_24V: C26.1, C27.1, F2.2, GLORY_24.1, GLORY_24.2, IC7.VS_1, IC7.VS_2, JMP1-0R.3, TIC0_7.9, TIC16_23.9, TIC8_15.9
- new net N$13: FM_RS.1, IC1G$1.R2OUT
- new net N$14: OK1.C, R34.1
- new net N$17: OK2.C, R37.1
- new net VPOWER: IC5.VPWR, JMP1-0R.2
- net PC_RX2: now also FM_RS.2, OK1.EMI, R36.2; no longer IC1G$1.R2OUT
- net PC_TX2: now also OK2.A
- net VDD: now also C36.1, JMP1-0R.1, OK1.COL; no longer IC5.VPWR
- net VSS: now also C36.2, R36.1, R37.2
