File: secs_q84 v2.sch (EAGLE design)
At the start: 132 parts, among them IC1 MAX203ECWP, IC2 REF3440TIDBVR, IC3 ADP151AUJZ-3.3-R7, IC4 ADM3095EBRZ, IC5 MCZ33996EK, IC6 74HC125D, IC7 TIC12400DCPR, IC8 PIC18F57Q84-I_PT

Commit message: up
Parts:
- R20, R21, R22, R23, R24: value 0ohm -> 56ohm
Connections:
- net PC_RX2: now also PVP_0.3
- net PC_TX2: now also PVP_0.8
Changed lines of the file:
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@@
 <part name="VSS53" library="supply1" library_urn="urn:adsk.eagle:library:371" deviceset="VSS" device=""/>
 <part name="VSS54" library="supply1" library_urn="urn:adsk.eagle:library:371" deviceset="VSS" device=""/>
-<part name="R20" library="rcl" library_urn="urn:adsk.eagle:library:334" deviceset="R-US_" device="R0805" package3d_urn="urn:adsk.eagle:package:23553/2" value="0ohm"/>
-<part name="R21" library="rcl" library_urn="urn:adsk.eagle:library:334" deviceset="R-US_" device="R0805" package3d_urn="urn:adsk.eagle:package:23553/2" value="0ohm"/>
-<part name="R22" library="rcl" library_urn="urn:adsk.eagle:library:334" deviceset="R-US_" device="R0805" package3d_urn="urn:adsk.eagle:package:23553/2" value="0ohm"/>
-<part name="R23" library="rcl" library_urn="urn:adsk.eagle:library:334" deviceset="R-US_" device="R0805" package3d_urn="urn:adsk.eagle:package:23553/2" value="0ohm"/>
-<part name="R24" library="rcl" library_urn="urn:adsk.eagle:library:334" deviceset="R-US_" device="R0805" package3d_urn="urn:adsk.eagle:package:23553/2" value="0ohm"/>
+<part name="R20" library="rcl" library_urn="urn:adsk.eagle:library:334" deviceset="R-US_" device="R0805" package3d_urn="urn:adsk.eagle:package:23553/2" value="56ohm"/>
+<part name="R21" library="rcl" library_urn="urn:adsk.eagle:library:334" deviceset="R-US_" device="R0805" package3d_urn="urn:adsk.eagle:package:23553/2" value="56ohm"/>
+<part name="R22" library="rcl" library_urn="urn:adsk.eagle:library:334" deviceset="R-US_" device="R0805" package3d_urn="urn:adsk.eagle:package:23553/2" value="56ohm"/>
+<part name="R23" library="rcl" library_urn="urn:adsk.eagle:library:334" deviceset="R-US_" device="R0805" package3d_urn="urn:adsk.eagle:package:23553/2" value="56ohm"/>
+<part name="R24" library="rcl" library_urn="urn:adsk.eagle:library:334" deviceset="R-US_" device="R0805" package3d_urn="urn:adsk.eagle:package:23553/2" value="56ohm"/>
 <part name="IC5" library="MCZ33996EK" deviceset="MCZ33996EK" device=""/>
 <part name="VSS14" library="supply1" library_urn="urn:adsk.eagle:library:371" deviceset="VSS" device=""/>
@@
 </instance>
 <instance part="R20" gate="G$1" x="139.7" y="25.4" smashed="yes">
-<attribute name="NAME" x="135.89" y="26.8986" size="1.778" layer="95"/>
-<attribute name="VALUE" x="135.89" y="22.098" size="1.778" layer="96"/>
+<attribute name="NAME" x="110.49" y="24.3586" size="1.778" layer="95"/>
+<attribute name="VALUE" x="118.11" y="24.638" size="1.778" layer="96"/>
 </instance>
 <instance part="R21" gate="G$1" x="139.7" y="22.86" smashed="yes">
-<attribute name="NAME" x="135.89" y="24.3586" size="1.778" layer="95"/>
-<attribute name="VALUE" x="135.89" y="19.558" size="1.778" layer="96"/>
+<attribute name="NAME" x="110.49" y="21.8186" size="1.778" layer="95"/>
+<attribute name="VALUE" x="118.11" y="22.098" size="1.778" layer="96"/>
 </instance>
 <instance part="R22" gate="G$1" x="139.7" y="20.32" smashed="yes">
-<attribute name="NAME" x="135.89" y="21.8186" size="1.778" layer="95"/>
-<attribute name="VALUE" x="135.89" y="17.018" size="1.778" layer="96"/>
+<attribute name="NAME" x="110.49" y="19.2786" size="1.778" layer="95"/>
+<attribute name="VALUE" x="118.11" y="19.558" size="1.778" layer="96"/>
 </instance>
 <instance part="R23" gate="G$1" x="139.7" y="17.78" smashed="yes">
-<attribute name="NAME" x="135.89" y="19.2786" size="1.778" layer="95"/>
-<attribute name="VALUE" x="135.89" y="14.478" size="1.778" layer="96"/>
+<attribute name="NAME" x="110.49" y="16.7386" size="1.778" layer="95"/>
+<attribute name="VALUE" x="118.11" y="17.018" size="1.778" layer="96"/>
 </instance>
 <instance part="R24" gate="G$1" x="139.7" y="15.24" smashed="yes">
-<attribute name="NAME" x="135.89" y="16.7386" size="1.778" layer="95"/>
-<attribute name="VALUE" x="135.89" y="11.938" size="1.778" layer="96"/>
+<attribute name="NAME" x="110.49" y="14.1986" size="1.778" layer="95"/>
+<attribute name="VALUE" x="118.11" y="14.478" size="1.778" layer="96"/>
 </instance>
 <instance part="IC5" gate="G$1" x="78.74" y="-53.34" smashed="yes">
@@
 <label x="393.7" y="-129.54" size="1.778" layer="95"/>
 </segment>
+<segment>
+<wire x1="45.72" y1="7.62" x2="33.02" y2="7.62" width="0.1524" layer="91"/>
+<pinref part="PVP_0" gate="G$1" pin="3"/>
+<junction x="45.72" y="7.62"/>
+<junction x="33.02" y="7.62"/>
+<label x="35.56" y="7.62" size="1.778" layer="95"/>
+</segment>
 </net>
 <net name="SS2" class="0">
@@
 <label x="393.7" y="-137.16" size="1.778" layer="95"/>
 </segment>
+<segment>
+<wire x1="68.58" y1="7.62" x2="81.28" y2="7.62" width="0.1524" layer="91"/>
+<pinref part="PVP_0" gate="G$1" pin="8"/>
+<junction x="68.58" y="7.62"/>
+<junction x="81.28" y="7.62"/>
+<label x="71.12" y="7.62" size="1.778" layer="95"/>
+</segment>
 </net>
 <net name="ANA4" class="0">
@@
 <label x="91.44" y="25.4" size="1.778" layer="95"/>
 <junction x="99.06" y="25.4"/>
-<label x="106.68" y="25.4" size="1.778" layer="95"/>
 <junction x="86.36" y="25.4"/>
 </segment>

Commit message: up
Changed lines of the file:
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@@
 </instance>
 <instance part="P+3" gate="VCC" x="55.88" y="73.66" smashed="yes" rot="R90">
-<attribute name="VALUE" x="58.42" y="71.12" size="1.778" layer="96" rot="R180"/>
+<attribute name="VALUE" x="53.34" y="73.66" size="1.778" layer="96" rot="R180"/>
 </instance>
 <instance part="FRAME1" gate="G$1" x="-142.24" y="-223.52" smashed="yes"/>

Commit message: update board to 1.308
Parts:
- added LED5: FM80 POWER, led:LEDCHIP-LED0603
- added R38: 10k, rcl:R-US_R0805
- renumbered JMP1 to VDD-TIC
Connections:
- new net N$15: LED5.A, R38.2
- net 0V: now also LED5.C
- net FM80_24: now also R38.1
Changed lines of the file:
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@@
 <part name="VSS86" library="supply1" library_urn="urn:adsk.eagle:library:371" deviceset="VSS" device=""/>
 <part name="VSS87" library="supply1" library_urn="urn:adsk.eagle:library:371" deviceset="VSS" device=""/>
-<part name="JMP1" library="jump-0r-smd" library_urn="urn:adsk.eagle:library:251" deviceset="0R-JUMP" device="A" package3d_urn="urn:adsk.eagle:package:15385/1"/>
+<part name="VDD-TIC" library="jump-0r-smd" library_urn="urn:adsk.eagle:library:251" deviceset="0R-JUMP" device="A" package3d_urn="urn:adsk.eagle:package:15385/1"/>
 <part name="VDD32" library="supply1" library_urn="urn:adsk.eagle:library:371" deviceset="VDD" device=""/>
 <part name="VDD18" library="supply1" library_urn="urn:adsk.eagle:library:371" deviceset="VDD" device=""/>
@@
 <part name="GND4" library="supply1" library_urn="urn:adsk.eagle:library:371" deviceset="0V" device=""/>
 <part name="FM_RS" library="jumper" library_urn="urn:adsk.eagle:library:252" deviceset="SJ" device="" package3d_urn="urn:adsk.eagle:package:15471/1" value="FM_RS"/>
+<part name="LED5" library="led" library_urn="urn:adsk.eagle:library:259" deviceset="LED" device="CHIP-LED0603" package3d_urn="urn:adsk.eagle:package:15819/3" value="FM80 POWER"/>
+<part name="R38" library="rcl" library_urn="urn:adsk.eagle:library:334" deviceset="R-US_" device="R0805" package3d_urn="urn:adsk.eagle:package:23553/2" value="10k"/>
+<part name="GND5" library="supply1" library_urn="urn:adsk.eagle:library:371" deviceset="0V" device=""/>
 </parts>
 <sheets>
@@
 <attribute name="VALUE" x="261.62" y="-213.36" size="1.778" layer="96" rot="R270"/>
 </instance>
-<instance part="JMP1" gate="-0R" x="53.34" y="-45.72" smashed="yes">
+<instance part="VDD-TIC" gate="-0R" x="53.34" y="-45.72" smashed="yes">
 <attribute name="NAME" x="53.34" y="-39.37" size="1.778" layer="95"/>
 </instance>
-<instance part="JMP1" gate="G$2" x="58.42" y="-40.64" smashed="yes"/>
+<instance part="VDD-TIC" gate="G$2" x="58.42" y="-40.64" smashed="yes"/>
 <instance part="VDD32" gate="G$1" x="50.8" y="-43.18" smashed="yes" rot="R90">
 <attribute name="VALUE" x="45.72" y="-40.64" size="1.778" layer="96" rot="R270"/>
@@
 <attribute name="VALUE" x="276.86" y="64.77" size="1.778" layer="96"/>
 </instance>
+<instance part="LED5" gate="G$1" x="398.78" y="-93.98" smashed="yes">
+<attribute name="NAME" x="390.652" y="-95.504" size="1.778" layer="95" rot="R180"/>
+<attribute name="VALUE" x="393.192" y="-93.345" size="1.778" layer="96" rot="R180"/>
+</instance>
+<instance part="R38" gate="G$1" x="398.78" y="-86.36" smashed="yes" rot="R270">
+<attribute name="NAME" x="400.2786" y="-82.55" size="1.778" layer="95" rot="R270"/>
+<attribute name="VALUE" x="395.478" y="-82.55" size="1.778" layer="96" rot="R270"/>
+</instance>
+<instance part="GND5" gate="1" x="398.78" y="-101.6" smashed="yes">
+<attribute name="VALUE" x="396.875" y="-104.14" size="1.778" layer="96"/>
+</instance>
 </instances>
 <busses>
@@
 </segment>
 <segment>
-<pinref part="JMP1" gate="-0R" pin="1"/>
+<pinref part="VDD-TIC" gate="-0R" pin="1"/>
 <pinref part="VDD32" gate="G$1" pin="VDD"/>
 <junction x="53.34" y="-43.18"/>
@@
 <segment>
 <wire x1="45.72" y1="-48.26" x2="53.34" y2="-48.26" width="0.1524" layer="91"/>
-<pinref part="JMP1" gate="-0R" pin="3"/>
+<pinref part="VDD-TIC" gate="-0R" pin="3"/>
 <junction x="45.72" y="-48.26"/>
 <junction x="53.34" y="-48.26"/>
@@
 <net name="VPOWER" class="1">
 <segment>
-<pinref part="JMP1" gate="-0R" pin="2"/>
+<pinref part="VDD-TIC" gate="-0R" pin="2"/>
 <wire x1="55.88" y1="-45.72" x2="58.42" y2="-45.72" width="0.1524" layer="91"/>
 <wire x1="58.42" y1="-45.72" x2="58.42" y2="-66.04" width="0.1524" layer="91"/>
@@
 <label x="330.2" y="-91.44" size="1.778" layer="95"/>
 </segment>
+<segment>
+<pinref part="LED5" gate="G$1" pin="C"/>
+<pinref part="GND5" gate="1" pin="0V"/>
+<junction x="398.78" y="-99.06"/>
+</segment>
 </net>
 <net name="FM80_24" class="0">
@@
 <label x="330.2" y="-93.98" size="1.778" layer="95"/>
 </segment>
+<segment>
+<wire x1="398.78" y1="-81.28" x2="398.78" y2="-68.58" width="0.1524" layer="91"/>
+<pinref part="R38" gate="G$1" pin="1"/>
+<junction x="398.78" y="-81.28"/>
+<junction x="398.78" y="-68.58"/>
+<label x="386.08" y="-73.66" size="1.778" layer="95"/>
+</segment>
 </net>
 <net name="N$13" class="0">
@@
 </segment>
 </net>
+<net name="N$15" class="0">
+<segment>
+<pinref part="LED5" gate="G$1" pin="A"/>
+<pinref part="R38" gate="G$1" pin="2"/>
+<junction x="398.78" y="-91.44"/>
+</segment>
+</net>

Commit message: cal analog inputs
Parts:
- renumbered LED1 to LED1_RED
Changed lines of the file:
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@@
 <part name="MISC_IO" library="con-lstb" library_urn="urn:adsk.eagle:library:162" deviceset="MA10-1" device="" package3d_urn="urn:adsk.eagle:package:8346/1" value="misc-io"/>
 <part name="VSS26" library="supply1" library_urn="urn:adsk.eagle:library:371" deviceset="VSS" device=""/>
-<part name="LED1" library="led" library_urn="urn:adsk.eagle:library:259" deviceset="LED" device="CHIPLED_0805" package3d_urn="urn:adsk.eagle:package:15821/2" value="L1"/>
+<part name="LED1_RED" library="led" library_urn="urn:adsk.eagle:library:259" deviceset="LED" device="CHIPLED_0805" package3d_urn="urn:adsk.eagle:package:15821/2" value="L1"/>
 <part name="LED2" library="led" library_urn="urn:adsk.eagle:library:259" deviceset="LED" device="CHIPLED_0805" package3d_urn="urn:adsk.eagle:package:15821/2" value="L2"/>
 <part name="LED3" library="led" library_urn="urn:adsk.eagle:library:259" deviceset="LED" device="CHIPLED_0805" package3d_urn="urn:adsk.eagle:package:15821/2" value="L3"/>
@@
 <attribute name="VALUE" x="0" y="22.86" size="1.778" layer="96" rot="R270"/>
 </instance>
-<instance part="LED1" gate="G$1" x="129.54" y="60.96" smashed="yes">
-<attribute name="NAME" x="133.096" y="56.388" size="1.778" layer="95" rot="R90"/>
+<instance part="LED1_RED" gate="G$1" x="129.54" y="60.96" smashed="yes">
+<attribute name="NAME" x="125.476" y="56.388" size="1.778" layer="95" rot="R90"/>
 <attribute name="VALUE" x="135.255" y="56.388" size="1.778" layer="96" rot="R90"/>
 </instance>
@@
 </segment>
 <segment>
-<pinref part="LED1" gate="G$1" pin="C"/>
+<pinref part="LED1_RED" gate="G$1" pin="C"/>
 <pinref part="VSS28" gate="G$1" pin="VSS"/>
 <junction x="129.54" y="55.88"/>
@@
 <net name="N$4" class="0">
 <segment>
-<pinref part="LED1" gate="G$1" pin="A"/>
+<pinref part="LED1_RED" gate="G$1" pin="A"/>
 <pinref part="R7" gate="G$1" pin="1"/>
 <junction x="129.54" y="63.5"/>

Commit message: add new code for serial interfaces
Connections:
- net DE3: no longer MODBUS.6
- net DERE: now also MODBUS.6
Changed lines of the file:
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@@
 <junction x="203.2" y="-30.48"/>
+</segment>
+<segment>
+<wire x1="279.4" y1="-20.32" x2="279.4" y2="-33.02" width="0.1524" layer="91"/>
+<pinref part="MODBUS" gate="1" pin="6"/>
+<junction x="279.4" y="-33.02"/>
+<junction x="279.4" y="-20.32"/>
+<label x="281.94" y="-27.94" size="1.778" layer="95"/>
 </segment>
 </net>
@@
 </segment>
 <segment>
-<wire x1="279.4" y1="-33.02" x2="279.4" y2="-20.32" width="0.1524" layer="91"/>
-<pinref part="MODBUS" gate="1" pin="6"/>
-<junction x="279.4" y="-20.32"/>
-<junction x="279.4" y="-33.02"/>
-<label x="281.94" y="-30.48" size="1.778" layer="95" rot="R90"/>
-</segment>
-<segment>

Commit message: up
Parts:
- R28, R29: value 400 ohm -> 390 ohm
Changed lines of the file:
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@@
 <part name="C28" library="rcl" library_urn="urn:adsk.eagle:library:334" deviceset="C-US" device="C0805" package3d_urn="urn:adsk.eagle:package:23617/2" value="0.1uf"/>
 <part name="VSS70" library="supply1" library_urn="urn:adsk.eagle:library:371" deviceset="VSS" device=""/>
-<part name="R28" library="rcl" library_urn="urn:adsk.eagle:library:334" deviceset="R-US_" device="R0805" package3d_urn="urn:adsk.eagle:package:23553/2" value="400 ohm"/>
-<part name="R29" library="rcl" library_urn="urn:adsk.eagle:library:334" deviceset="R-US_" device="R0805" package3d_urn="urn:adsk.eagle:package:23553/2" value="400 ohm"/>
+<part name="R28" library="rcl" library_urn="urn:adsk.eagle:library:334" deviceset="R-US_" device="R0805" package3d_urn="urn:adsk.eagle:package:23553/2" value="390 ohm"/>
+<part name="R29" library="rcl" library_urn="urn:adsk.eagle:library:334" deviceset="R-US_" device="R0805" package3d_urn="urn:adsk.eagle:package:23553/2" value="390 ohm"/>
 <part name="TIC_DIGITAL" library="con-lstb" library_urn="urn:adsk.eagle:library:162" deviceset="MA04-1" device="" package3d_urn="urn:adsk.eagle:package:8337/1" value="TIC_DIGITAL"/>
 <part name="VSS71" library="supply1" library_urn="urn:adsk.eagle:library:371" deviceset="VSS" device=""/>

Commit message: up
Parts:
- added R39: 120, rcl:R-US_R0805
- R20, R21, R22, R23, R24: value 56ohm -> 22 ohm
Connections:
- net +3V3: now also R39.2
- net VSS: now also R39.1
Changed lines of the file:
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@@
 <part name="VSS53" library="supply1" library_urn="urn:adsk.eagle:library:371" deviceset="VSS" device=""/>
 <part name="VSS54" library="supply1" library_urn="urn:adsk.eagle:library:371" deviceset="VSS" device=""/>
-<part name="R20" library="rcl" library_urn="urn:adsk.eagle:library:334" deviceset="R-US_" device="R0805" package3d_urn="urn:adsk.eagle:package:23553/2" value="56ohm"/>
-<part name="R21" library="rcl" library_urn="urn:adsk.eagle:library:334" deviceset="R-US_" device="R0805" package3d_urn="urn:adsk.eagle:package:23553/2" value="56ohm"/>
-<part name="R22" library="rcl" library_urn="urn:adsk.eagle:library:334" deviceset="R-US_" device="R0805" package3d_urn="urn:adsk.eagle:package:23553/2" value="56ohm"/>
-<part name="R23" library="rcl" library_urn="urn:adsk.eagle:library:334" deviceset="R-US_" device="R0805" package3d_urn="urn:adsk.eagle:package:23553/2" value="56ohm"/>
-<part name="R24" library="rcl" library_urn="urn:adsk.eagle:library:334" deviceset="R-US_" device="R0805" package3d_urn="urn:adsk.eagle:package:23553/2" value="56ohm"/>
+<part name="R20" library="rcl" library_urn="urn:adsk.eagle:library:334" deviceset="R-US_" device="R0805" package3d_urn="urn:adsk.eagle:package:23553/2" value="22 ohm"/>
+<part name="R21" library="rcl" library_urn="urn:adsk.eagle:library:334" deviceset="R-US_" device="R0805" package3d_urn="urn:adsk.eagle:package:23553/2" value="22 ohm"/>
+<part name="R22" library="rcl" library_urn="urn:adsk.eagle:library:334" deviceset="R-US_" device="R0805" package3d_urn="urn:adsk.eagle:package:23553/2" value="22 ohm"/>
+<part name="R23" library="rcl" library_urn="urn:adsk.eagle:library:334" deviceset="R-US_" device="R0805" package3d_urn="urn:adsk.eagle:package:23553/2" value="22 ohm"/>
+<part name="R24" library="rcl" library_urn="urn:adsk.eagle:library:334" deviceset="R-US_" device="R0805" package3d_urn="urn:adsk.eagle:package:23553/2" value="22 ohm"/>
 <part name="IC5" library="MCZ33996EK" deviceset="MCZ33996EK" device=""/>
 <part name="VSS14" library="supply1" library_urn="urn:adsk.eagle:library:371" deviceset="VSS" device=""/>
@@
 <part name="R38" library="rcl" library_urn="urn:adsk.eagle:library:334" deviceset="R-US_" device="R0805" package3d_urn="urn:adsk.eagle:package:23553/2" value="10k"/>
 <part name="GND5" library="supply1" library_urn="urn:adsk.eagle:library:371" deviceset="0V" device=""/>
+<part name="R39" library="rcl" library_urn="urn:adsk.eagle:library:334" deviceset="R-US_" device="R0805" package3d_urn="urn:adsk.eagle:package:23553/2" value="120"/>
+<part name="VSS91" library="supply1" library_urn="urn:adsk.eagle:library:371" deviceset="VSS" device=""/>
 </parts>
 <sheets>
@@
 <attribute name="VALUE" x="396.875" y="-104.14" size="1.778" layer="96"/>
 </instance>
+<instance part="R39" gate="G$1" x="322.58" y="-60.96" smashed="yes" rot="R90">
+<attribute name="NAME" x="321.0814" y="-64.77" size="1.778" layer="95" rot="R90"/>
+<attribute name="VALUE" x="325.882" y="-64.77" size="1.778" layer="96" rot="R90"/>
+</instance>
+<instance part="VSS91" gate="G$1" x="322.58" y="-68.58" smashed="yes">
+<attribute name="VALUE" x="330.2" y="-66.04" size="1.778" layer="96" rot="R180"/>
+</instance>
 </instances>
 <busses>
@@
 <pinref part="C16" gate="G$1" pin="2"/>
 <pinref part="VSS40" gate="G$1" pin="VSS"/>
+<junction x="332.74" y="-63.5"/>
 </segment>
 <segment>
 <pinref part="C17" gate="G$1" pin="2"/>
 <pinref part="VSS41" gate="G$1" pin="VSS"/>
+<junction x="340.36" y="-63.5"/>
 </segment>
 <segment>
@@
 <junction x="388.62" y="-116.84"/>
 </segment>
+<segment>
+<pinref part="R39" gate="G$1" pin="1"/>
+<pinref part="VSS91" gate="G$1" pin="VSS"/>
+<junction x="322.58" y="-66.04"/>
+</segment>
 </net>
 <net name="CPU_CLK" class="0">
@@
 <junction x="332.74" y="-55.88"/>
 <junction x="340.36" y="-55.88"/>
+<pinref part="R39" gate="G$1" pin="2"/>
+<wire x1="322.58" y1="-55.88" x2="332.74" y2="-55.88" width="0.1524" layer="91"/>
+<junction x="322.58" y="-55.88"/>
 </segment>
 <segment>

Commit message: up
Parts:
- R19, R7, R8, R9: value 1k -> 2.2k
Changed lines of the file:
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@@
 <part name="VSS29" library="supply1" library_urn="urn:adsk.eagle:library:371" deviceset="VSS" device=""/>
 <part name="VSS30" library="supply1" library_urn="urn:adsk.eagle:library:371" deviceset="VSS" device=""/>
-<part name="R7" library="rcl" library_urn="urn:adsk.eagle:library:334" deviceset="R-US_" device="R0805" package3d_urn="urn:adsk.eagle:package:23553/2" value="1k"/>
-<part name="R8" library="rcl" library_urn="urn:adsk.eagle:library:334" deviceset="R-US_" device="R0805" package3d_urn="urn:adsk.eagle:package:23553/2" value="1k"/>
-<part name="R9" library="rcl" library_urn="urn:adsk.eagle:library:334" deviceset="R-US_" device="R0805" package3d_urn="urn:adsk.eagle:package:23553/2" value="1k"/>
+<part name="R7" library="rcl" library_urn="urn:adsk.eagle:library:334" deviceset="R-US_" device="R0805" package3d_urn="urn:adsk.eagle:package:23553/2" value="2.2k"/>
+<part name="R8" library="rcl" library_urn="urn:adsk.eagle:library:334" deviceset="R-US_" device="R0805" package3d_urn="urn:adsk.eagle:package:23553/2" value="2.2k"/>
+<part name="R9" library="rcl" library_urn="urn:adsk.eagle:library:334" deviceset="R-US_" device="R0805" package3d_urn="urn:adsk.eagle:package:23553/2" value="2.2k"/>
 <part name="TP1" library="testpad" library_urn="urn:adsk.eagle:library:385" deviceset="PTR1" device="PAD1-13" package3d_urn="urn:adsk.eagle:package:27946/1"/>
 <part name="RESET" library="jumper" library_urn="urn:adsk.eagle:library:252" deviceset="SJ" device="" package3d_urn="urn:adsk.eagle:package:15471/1" value="reset"/>
@@
 <part name="R18" library="rcl" library_urn="urn:adsk.eagle:library:334" deviceset="R-US_" device="R0805" package3d_urn="urn:adsk.eagle:package:23553/2" value="0ohm"/>
 <part name="VSS50" library="supply1" library_urn="urn:adsk.eagle:library:371" deviceset="VSS" device=""/>
-<part name="R19" library="rcl" library_urn="urn:adsk.eagle:library:334" deviceset="R-US_" device="R0805" package3d_urn="urn:adsk.eagle:package:23553/2" value="1k"/>
+<part name="R19" library="rcl" library_urn="urn:adsk.eagle:library:334" deviceset="R-US_" device="R0805" package3d_urn="urn:adsk.eagle:package:23553/2" value="2.2k"/>
 <part name="LED4" library="led" library_urn="urn:adsk.eagle:library:259" deviceset="LED" device="CHIP-LED0603" package3d_urn="urn:adsk.eagle:package:15819/3" value="POWER"/>
 <part name="VSS2" library="supply1" library_urn="urn:adsk.eagle:library:371" deviceset="VSS" device=""/>
@@
 </instance>
 <instance part="C18" gate="G$1" x="320.04" y="-27.94" smashed="yes">
-<attribute name="NAME" x="321.056" y="-27.305" size="1.778" layer="95"/>
+<attribute name="NAME" x="313.436" y="-32.385" size="1.778" layer="95"/>
 <attribute name="VALUE" x="323.596" y="-32.131" size="1.778" layer="96"/>
 </instance>
 <instance part="C19" gate="G$1" x="327.66" y="-27.94" smashed="yes">
-<attribute name="NAME" x="328.676" y="-27.305" size="1.778" layer="95"/>
+<attribute name="NAME" x="328.676" y="-34.925" size="1.778" layer="95"/>
 <attribute name="VALUE" x="328.676" y="-32.131" size="1.778" layer="96"/>
 </instance>
